File: PDB/PDB_MH.sch (EAGLE design)
At the start: 23 parts

Commit message: Add battery buzzer to board
Parts:
- added JP1: XH_CONN, pie:XH_CONNECTOR_4POS
- added JP2: (no value), pie:M02PTH
- added LED1: RED, pie:LED0805
- added LED2: 7-SEGMENT, pie:7-SEGMENT-4DIGIT-YOUNGSUN
- added LS1: BUZZER, pie:BUZZER
- added Q1, Q2: IRFML8244, pie:N-CHANNEL-MOSFETSOT23-3
- added Q3: PMOSFET, pie:P-CHANNEL-MOSFETSOT23-3
- added Q4, Q5: P-CHANNEL-MOSFETSOT23-3, pie:P-CHANNEL-MOSFETSOT23-3
- added R1, R10, R16, R2, R5, R6, R7, R8: 10k, pie:R-US_R0603
- added R11: 130, pie:R-US_R0603
- added R12, R13, R14, R15: 330, pie:R-US_R0603
- added R3: 30k, pie:R-US_R0603
- added R4: 51k, pie:R-US_R0603
- added R9: 100, pie:R-US_R0603
- added S1, S2: DPST_SWITCH, pie:DPST_SWITCH
- added SJ1: GND to BGND, pie:SOLDERJUMPERNO
- added UC1: ARDUINO_PRO_MICRO, pie:ARDUINO_PRO_MICRO
- renumbered U$1 to XT60
Connections:
- new net A: LED2.A, UC1.8
- new net B: LED2.B, UC1.9
- new net BCELL1: JP1.2, Q3.S
- new net BCELL2: JP1.3, Q4.S
- new net BCELL3: JP1.4, Q5.S, R1.2, S1.P1
- new net BGND: JP1.1, S1.P2, SJ1.1
- new net BUZZER_SIGNAL: R11.2, R9.1, UC1.A3
- new net C: LED2.C, UC1.7
- new net CALIB: R16.1, S2.P1', S2.P2', UC1.10
- new net D: LED2.D, UC1.2
- new net DIG_1: R12.2, UC1.6
- new net DIG_2: R13.2, UC1.5
- new net DIG_3: R14.2, UC1.4
- new net DIG_4: R15.2, UC1.3
- new net DIV_EN: Q2.G, R8.2, UC1.16
- new net DP: LED2.DP, UC1.TXO
- new net E: LED2.E, UC1.RXI
- new net F: LED2.F, UC1.15
- new net G: LED2.G, UC1.14
- new net IO0: R2.1, R5.2, UC1.A0
- new net IO1: R3.1, R6.2, UC1.A1
- new net IO2: R4.1, R7.2, UC1.A2
- new net N$1: Q2.D, Q3.G, Q4.G, Q5.G, R1.1
- new net N$11: LED2.DIG2, R13.1
- new net N$13: LED2.DIG3, R14.1
- new net N$15: LED2.DIG4, R15.1
- new net N$2: Q3.D, R2.2
- new net N$3: Q4.D, R3.2
- new net N$4: Q5.D, R4.2
- new net N$5: LS1.C, Q1.D
- new net N$6: Q1.G, R10.2, R9.2
- new net N$7: LED1.A, R11.1
- new net N$9: LED2.DIG1, R12.1
- new net RAW: S1.P1', UC1.RAW
- net 5V: now also LS1.A, S2.P1, S2.P2, UC1.VCC
- net GND: now also JP2.1, JP2.2, LED1.C, Q1.S@2, Q2.S@2, R10.1, R16.2, R5.1, R6.1, R7.1, R8.1, S1.P2', SJ1.2, UC1.GND@0, UC1.GND@1, UC1.GND@2
Other:
- note added: "8-SEG DISPLAY ARRAY"
- note added: "ARDUINO INTERFACE"
- note added: "BATTERY DISCONNECT"
- note added: "BATTERY INPUT"
- note added: "BUZZER CIRCUIT"
- note added: "CALIBRATION BUTTON"
- note added: "Connect BCELL3 to RAW, which will get regulated on the arduino."
- note added: "DEBUG FEATURES"
- note added: "LED CIRCUIT"
- note added: "RESISTOR DIVIDERS"
- note added: "SECONDARY POWER"
- note added: "Use high-precision (better than 0.5%) resistors"
