File: TeamFlag/TeamFlag.brd (EAGLE design)
At the start: 40.6 x 44.5 mm, 24 parts, among them IC1 ARDUINO_PRO_MICROSMD, Q3 N-CH, Q4 N-CH

Commit message: Update teamflag
Connections:
- net GND: now also IC1.GND@2; no longer IC1.GND@3
Routing:
- net GND: track 10.7 -> 16.5 mm
- net YELLOW(IO2): track 27.1 -> 24.4 mm
- net BLUE(IO1): track 17.6 -> 15.8 mm
Other:
- board text added: "+"
Changed lines of the file:
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@@
 <setting verticaltext="up"/>
 </settings>
-<grid distance="0.05" unitdist="inch" unit="inch" style="lines" multiple="1" display="yes" altdistance="0.005" altunitdist="inch" altunit="inch"/>
+<grid distance="0.01" unitdist="inch" unit="inch" style="lines" multiple="1" display="yes" altdistance="0.005" altunitdist="inch" altunit="inch"/>
 <layers>
 <layer number="1" name="Top" color="4" fill="1" visible="yes" active="yes"/>
@@
 <layer number="251" name="SMDround" color="12" fill="11" visible="no" active="no"/>
 <layer number="254" name="cooling" color="7" fill="1" visible="yes" active="yes"/>
-<layer number="255" name="routoute" color="7" fill="1" visible="no" active="yes"/>
+<layer number="255" name="routoute" color="7" fill="1" visible="yes" active="yes"/>
 </layers>
 <board>
@@
 For more information, visit:
 https://github.com/pioneers/SmartSensors</text>
+<text x="2.794" y="35.56" size="1.778" layer="22" rot="MR0" align="center">+</text>
+<text x="9.144" y="39.624" size="1.778" layer="22" rot="MR0" align="center">+</text>
+<text x="36.068" y="37.084" size="1.778" layer="22" rot="MR0" align="center">+</text>
+<text x="39.37" y="33.274" size="1.778" layer="22" rot="MR0" align="center">+</text>
 </plain>
 <attributes>
@@
 </element>
 <element name="R1" library="pie" package="R0603" value="200" x="30.988" y="16.891" smashed="yes" rot="R90">
-<attribute name="NAME" x="30.099" y="14.7828" size="0.762" layer="25" font="vector" ratio="15" rot="R90"/>
-<attribute name="VALUE" value="&gt;VALUE" x="30.1752" y="16.3068" size="0.762" layer="27" font="vector" ratio="15" rot="R270" align="top-right"/>
 <attribute name="MANUFACTURER" value="Rohm Semiconductor" x="30.988" y="16.891" size="1.778" layer="27" rot="R90" display="off"/>
 <attribute name="DISTRIBUTOR" value="DigiKey" x="30.988" y="16.891" size="1.778" layer="27" rot="R90" display="off"/>
@@
 <attribute name="MANUFACTURER_PART_NUMBER" value="" x="30.988" y="16.891" size="1.778" layer="27" rot="R90" display="off"/>
 <attribute name="DESCRIPTION" value="RESISTOR, American symbol" x="30.988" y="16.891" size="1.778" layer="27" rot="R90" display="off"/>
+<attribute name="NAME" x="29.718" y="17.78" size="0.762" layer="25" font="vector" ratio="10" rot="R90"/>
+<attribute name="VALUE" x="32.766" y="17.78" size="0.762" layer="27" font="vector" rot="R90"/>
 </element>
 <element name="R2" library="pie" package="R0603" value="200" x="12.192" y="17.145" smashed="yes" rot="R90">
@@
 <attribute name="VALUE" x="5.45880625" y="31.758984375" size="0.762" layer="26" font="vector" ratio="15" rot="MR309" align="center"/>
 </element>
-<element name="IC1" library="pie" package="ARDUINO_PRO_MICRO_SM" value="ARDUINO_PRO_MICROSMD" x="35.052" y="9.144" rot="R90"/>
+<element name="IC1" library="pie" package="ARDUINO_PRO_MICRO_SM" value="ARDUINO_PRO_MICROSMD" x="35.052" y="9.144" smashed="yes" rot="R90"/>
 <element name="Q3" library="pie" package="SOT23-3" value="N-CH" x="35.052" y="16.002" smashed="yes" rot="R90">
 <attribute name="NAME" x="33.147" y="14.732" size="1.27" layer="25" font="vector" ratio="10" rot="R90"/>
@@
 <signal name="YELLOW(IO2)">
 <contactref element="R4" pad="2"/>
-<wire x1="17.51" y1="8.0796" x2="19.2786" y2="6.311" width="0.4064" layer="1"/>
-<wire x1="19.2786" y1="6.311" x2="20.613" y2="6.311" width="0.4064" layer="1"/>
-<wire x1="20.613" y1="6.311" x2="21.336" y2="5.588" width="0.4064" layer="1"/>
-<wire x1="21.336" y1="5.588" x2="21.336" y2="3.81" width="0.4064" layer="1"/>
-<wire x1="21.336" y1="3.81" x2="22.098" y2="3.048" width="0.4064" layer="1"/>
-<wire x1="22.098" y1="3.048" x2="25.4" y2="3.048" width="0.4064" layer="1"/>
 <contactref element="IC1" pad="8"/>
-<wire x1="25.4" y1="3.048" x2="31.242" y2="8.89" width="0.4064" layer="1"/>
-<wire x1="31.242" y1="8.89" x2="31.242" y2="9.144" width="0.4064" layer="1"/>
 <contactref element="Q4" pad="1"/>
-<wire x1="18.272" y1="15.306" x2="17.51" y2="14.544" width="0.4064" layer="1"/>
-<wire x1="17.51" y1="14.544" x2="17.51" y2="8.0796" width="0.4064" layer="1"/>
+<wire x1="18.272" y1="15.306" x2="18.272" y2="12.208" width="0.4064" layer="1"/>
+<wire x1="18.272" y1="12.208" x2="20.32" y2="10.16" width="0.4064" layer="1"/>
+<wire x1="20.32" y1="10.16" x2="20.32" y2="7.3524" width="0.4064" layer="1"/>
+<wire x1="20.32" y1="7.3524" x2="19.2786" y2="6.311" width="0.4064" layer="1"/>
+<wire x1="31.242" y1="12.446" x2="28.382" y2="15.306" width="0.4064" layer="1"/>
+<wire x1="28.382" y1="15.306" x2="18.272" y2="15.306" width="0.4064" layer="1"/>
 </signal>
 <signal name="GND">
@@
 <vertex x="40.64" y="44.45"/>
 </polygon>
-<contactref element="IC1" pad="GND@3"/>
+<contactref element="IC1" pad="GND@2"/>
 <contactref element="IC1" pad="2"/>
 <contactref element="IC1" pad="3"/>
@@
 <contactref element="Q4" pad="2"/>
 <contactref element="R4" pad="1"/>
-<wire x1="2.8366875" y1="32.385721875" x2="5.250409375" y2="29.972" width="0.4064" layer="16"/>
-<wire x1="5.250409375" y1="29.972" x2="6.096" y2="29.972" width="0.4064" layer="16"/>
-<via x="6.096" y="29.972" extent="1-16" drill="0.5"/>
-<wire x1="6.096" y1="29.972" x2="8.382" y2="27.686" width="0.4064" layer="1"/>
-<wire x1="8.382" y1="27.686" x2="8.382" y2="24.513" width="0.4064" layer="1"/>
+<wire x1="2.8366875" y1="32.385721875" x2="2.8366875" y2="26.3733125" width="0.4064" layer="16"/>
+<wire x1="2.8366875" y1="26.3733125" x2="7.62" y2="21.59" width="0.4064" layer="16"/>
+<via x="7.62" y="21.59" extent="1-16" drill="0.5"/>
+<wire x1="7.62" y1="21.59" x2="8.597" y2="20.613" width="0.4064" layer="1"/>
+<wire x1="8.597" y1="20.613" x2="10.922" y2="20.613" width="0.4064" layer="1"/>
 </signal>
 <signal name="BLUE(IO1)">
 <contactref element="R3" pad="2"/>
-<wire x1="23.8506" y1="6.311" x2="23.8506" y2="9.1186" width="0.4064" layer="1"/>
-<wire x1="23.8506" y1="9.1186" x2="26.162" y2="11.43" width="0.4064" layer="1"/>
-<wire x1="26.162" y1="11.43" x2="27.94" y2="11.43" width="0.4064" layer="1"/>
 <contactref element="IC1" pad="7"/>
-<wire x1="28.702" y1="12.446" x2="28.702" y2="12.192" width="0.4064" layer="1"/>
-<wire x1="28.702" y1="12.192" x2="27.94" y2="11.43" width="0.4064" layer="1"/>
 <contactref element="Q3" pad="1"/>
-<wire x1="28.702" y1="12.446" x2="30.988" y2="12.446" width="0.4064" layer="1"/>
-<wire x1="30.988" y1="12.446" x2="32.512" y2="13.97" width="0.4064" layer="1"/>
-<wire x1="32.512" y1="13.97" x2="34.97" y2="13.97" width="0.4064" layer="1"/>
-<wire x1="34.97" y1="13.97" x2="36.052" y2="15.052" width="0.4064" layer="1"/>
+<wire x1="28.702" y1="9.144" x2="30.144" y2="9.144" width="0.4064" layer="1"/>
+<wire x1="30.144" y1="9.144" x2="36.052" y2="15.052" width="0.4064" layer="1"/>
+<wire x1="28.702" y1="9.144" x2="26.6836" y2="9.144" width="0.4064" layer="1"/>
+<wire x1="26.6836" y1="9.144" x2="23.8506" y2="6.311" width="0.4064" layer="1"/>
 </signal>
 <signal name="BSOURCE">
@@
 <wire x1="23.876" y1="22.86" x2="17.78" y2="22.86" width="0.4064" layer="16"/>
 <wire x1="17.78" y1="22.86" x2="15.24" y2="20.32" width="0.4064" layer="16"/>
-<wire x1="10.922" y1="22.313" x2="13.247" y2="22.313" width="0.4064" layer="1"/>
-<wire x1="13.247" y1="22.313" x2="15.24" y2="20.32" width="0.4064" layer="1"/>
-<wire x1="13.122" y1="24.513" x2="10.922" y2="22.313" width="0.4064" layer="1"/>
 <contactref element="IC1" pad="VCC"/>
-<wire x1="13.122" y1="24.513" x2="13.462" y2="24.513" width="0" layer="19" extent="1-1"/>
+<wire x1="13.462" y1="24.638" x2="11.137" y2="22.313" width="0.4064" layer="1"/>
+<wire x1="11.137" y1="22.313" x2="10.922" y2="22.313" width="0.4064" layer="1"/>
+<wire x1="11.137" y1="22.313" x2="13.13" y2="20.32" width="0.4064" layer="1"/>
+<wire x1="13.13" y1="20.32" x2="15.24" y2="20.32" width="0.4064" layer="1"/>
 </signal>
 <signal name="LED4">
@@
 <contactref element="IC1" pad="A3"/>
 <wire x1="13.169" y1="30.9" x2="16.002" y2="28.067" width="0.4064" layer="1"/>
-<wire x1="16.002" y1="28.067" x2="16.002" y2="27.813" width="0.4064" layer="1"/>
+<wire x1="16.002" y1="28.067" x2="16.002" y2="27.94" width="0.4064" layer="1"/>
 </signal>
 <signal name="LED1R">
@@
 <signal name="LED1">
 <contactref element="R5" pad="2"/>
-<wire x1="26.67" y1="30.9" x2="23.876" y2="28.106" width="0.4064" layer="1"/>
 <contactref element="IC1" pad="A0"/>
-<wire x1="23.622" y1="24.513" x2="23.876" y2="24.767" width="0.4064" layer="1"/>
-<wire x1="23.876" y1="24.767" x2="23.876" y2="28.106" width="0.4064" layer="1"/>
+<wire x1="23.622" y1="24.638" x2="23.622" y2="27.852" width="0.4064" layer="1"/>
+<wire x1="23.622" y1="27.852" x2="26.67" y2="30.9" width="0.4064" layer="1"/>
 </signal>
 <signal name="LED2">
@@
 <contactref element="IC1" pad="A1"/>
 <wire x1="21.59" y1="30.9" x2="21.082" y2="30.392" width="0.4064" layer="1"/>
-<wire x1="21.082" y1="30.392" x2="21.082" y2="27.813" width="0.4064" layer="1"/>
+<wire x1="21.082" y1="30.392" x2="21.082" y2="27.94" width="0.4064" layer="1"/>
 </signal>
 <signal name="LED3">
@@
 <contactref element="IC1" pad="A2"/>
 <wire x1="16.51" y1="30.9" x2="18.542" y2="28.868" width="0.4064" layer="1"/>
-<wire x1="18.542" y1="28.868" x2="18.542" y2="24.513" width="0.4064" layer="1"/>
+<wire x1="18.542" y1="28.868" x2="18.542" y2="24.638" width="0.4064" layer="1"/>
 </signal>
 </signals>
