File: Boards/BatteryBuzzer/Test_Board/Test_Board/test_board.brd (EAGLE design)
At the start: 0 parts

Commit message: ggetting caught up
Parts:
- added IC1: ARDUINO_PRO_MICRO, pie:ARDUINO_PRO_MICRO
- added R1, R2, R3, R4: >VALUE, pie:R0603
- added U$1: SN74HC4852, pie:DIL16
- added U$2: TL072, pie:DIL08
- added U$3: SOT-23_6PIN, pie:SOT-23_6PIN
- added U$4: XH_CONNECTOR_4POS, pie:XH_CONNECTOR_4POS_2.5MM

Commit message: SO MUCH
Parts:
- added R5, R6: 10k, pie:R0603
- added U$5: SN74HC4852, pie:DIL16
- R1, R2, R3, R4: value >VALUE -> 10k
- renumbered U$4 to BATTERY_CONNECT
Connections:
- new net 2-COM: R4.2, U$1.3
- new net 5V: IC1.RAW
- new net A: IC1.A1, U$1.10
- new net ADC_1-COM: U$3.P$1, U$5.13
- new net ADC_2-COM: U$3.P$4, U$5.3
- new net ADC_A: IC1.15, U$5.10
- new net ADC_B: IC1.14, U$5.9
- new net ADC_INH: IC1.16, U$5.6
- new net AMP-OUT: IC1.A3
- new net AMP_OUT: R3.1, U$2.1
- new net B: IC1.A0, U$1.9
- new net BCELL1: BATTERY_CONNECT.2, U$1.12, U$1.5, U$5.12, U$5.5
- new net BCELL2: BATTERY_CONNECT.3, U$1.14, U$1.2, U$5.14, U$5.2
- new net BCELL3: BATTERY_CONNECT.4, U$1.15, U$5.15
- new net GND: BATTERY_CONNECT.1, IC1.GND@0, IC1.GND@1, IC1.GND@2, R2.1, U$1.1, U$1.11, U$1.4, U$1.8, U$2.4, U$3.P$2, U$5.1, U$5.11, U$5.4, U$5.8
- new net INH_CONTROL: IC1.A2, U$1.6
- new net N$2: R1.2, R2.2, U$2.3
- new net N$3: R3.2, R4.1, U$2.2
- new net N$5: R1.1, U$1.13
- new net SCL: IC1.3, R6.1, U$3.P$3
- new net SDA: IC1.2, R5.1, U$3.P$6
- new net VCC: IC1.VCC, R5.2, R6.2, U$1.16, U$3.P$5, U$5.16

Commit message: Forgot to power the op amp
Connections:
- net BCELL3: now also U$2.8
Changed lines of the file:
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@@
 <contactref element="U$1" pad="15"/>
 <contactref element="U$5" pad="15"/>
+<contactref element="U$2" pad="8"/>
 <wire x1="-37.08999375" y1="-64.959990625" x2="-44.45" y2="-106.68" width="0" layer="19" extent="1-1"/>
-<wire x1="-40.64" y1="-19.05" x2="-37.08999375" y2="-64.959990625" width="0" layer="19" extent="1-1"/>
+<wire x1="-43.18" y1="-40.64" x2="-37.08999375" y2="-64.959990625" width="0" layer="19" extent="1-1"/>
+<wire x1="-40.64" y1="-19.05" x2="-43.18" y2="-40.64" width="0" layer="19" extent="1-1"/>
 </signal>
 <signal name="BCELL2">

Commit message: Started routing
Parts:
- added ADC_MUX_INPUTS, AMP_MUX_INPUTS, EXTERNAL_POWER: (no value), pie:1X02
- added LED1, LED2: GREEN, pie:LED-0603
- added OUTPUT_TEST_PINS: (no value), pie:1X03
- added R7, R8: 330, pie:R0603
- moved R6 170.0 mm to (53.3, 2.54)
- moved R3 168.7 mm to (40.6, 50.8), turned to 180 degrees
- moved BATTERY_CONNECT 164.4 mm to (78.7, 48.3)
- moved R5 161.8 mm to (48.3, 2.54), turned to 180 degrees
- moved U$5 143.8 mm to (31.8, 15.2), turned to 270 degrees
- moved R4 137.4 mm to (43.2, 2.54)
- moved R2 136.6 mm to (48.3, 8.89)
- moved R1 128.6 mm to (43.2, 8.89)
- moved U$2 126.9 mm to (55.9, 39.4), turned to 270 degrees
- moved U$3 125.0 mm to (45.7, 24.1), turned to 270 degrees
- moved U$1 90.7 mm to (31.8, 39.4), turned to 270 degrees
- moved IC1 73.0 mm to (21.6, 35.6), turned to 180 degrees
Connections:
- removed net N$5: R1.1, U$1.13
- new net 1-COM: AMP_MUX_INPUTS.2, R1.1, U$1.13
- new net ADC_OUT: IC1.6, OUTPUT_TEST_PINS.3
- new net LED_1: IC1.4, LED1.A
- new net LED_2: IC1.5, LED2.A
- new net N$7: LED2.C, R8.2
- new net N$8: LED1.C, R7.2
- net 2-COM: now also AMP_MUX_INPUTS.1
- net 5V: now also EXTERNAL_POWER.2
- net ADC_1-COM: now also ADC_MUX_INPUTS.2
- net ADC_2-COM: now also ADC_MUX_INPUTS.1
- net AMP_OUT: now also OUTPUT_TEST_PINS.2
- net GND: now also EXTERNAL_POWER.1, OUTPUT_TEST_PINS.1, R7.1, R8.1
Routing:
- net 5V: track 0.00 -> 48.3 mm
- added copper zone on layer 1, net GND
Other:
- board outline added: 92.7 x 54.6 mm

Commit message: Semi done routing
Parts:
- moved R2 47.2 mm to (22.6, 48.5), turned to 180 degrees
- moved R4 46.7 mm to (22.6, 44.5)
- moved R1 46.5 mm to (22.6, 50.5), turned to 180 degrees
- moved ADC_MUX_INPUTS 20.0 mm to (68.8, 10.9)
- moved AMP_MUX_INPUTS 19.9 mm to (68.8, 18.8)
- moved OUTPUT_TEST_PINS 19.8 mm to (68.8, 28.2)
- moved R3 18.5 mm to (22.6, 46.5)
- moved R7 12.2 mm to (46.2, 51.1)
- moved R8 11.4 mm to (48.3, 27.9)
- moved BATTERY_CONNECT 11.4 mm to (67.3, 48.3)
- moved U$2 3.05 mm to (52.8, 39.4)
- moved U$3 1.83 mm to (44.7, 25.7)
- moved R6 1.61 mm to (53.8, 4.06), turned to 180 degrees
- moved R5 1.52 mm to (48.3, 4.06)
- moved LED1 0.57 mm to (52.8, 51.1)
Connections:
- removed net AMP-OUT: IC1.A3
Routing:
- net BCELL2: track 0.00 -> 80.5 mm
- net BCELL1: track 0.00 -> 76.6 mm
- net ADC_A: track 0.00 -> 72.0 mm
- net ADC_B: track 0.00 -> 57.9 mm
- net ADC_INH: track 0.00 -> 55.0 mm
- net N$3: track 0.00 -> 47.4 mm
- net 1-COM: track 0.00 -> 45.2 mm, vias 0 -> 1
- net INH_CONTROL: track 0.00 -> 43.8 mm
- net N$2: track 0.00 -> 43.3 mm
- net VCC: track 0.00 -> 33.2 mm
- net AMP_OUT: track 0.00 -> 29.6 mm
- net ADC_1-COM: track 0.00 -> 27.4 mm
- net SCL: track 0.00 -> 22.4 mm
- net SDA: track 0.00 -> 21.2 mm
- net BCELL3: track 0.00 -> 18.1 mm
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Other:
- board size 92.7 x 54.6 mm -> 81.3 x 54.6 mm

Commit message: Finished
Parts:
- removed ADC_MUX_INPUTS, AMP_MUX_INPUTS: (no value), pie:1X02
- removed LED1, LED2: GREEN, pie:LED-0603
- removed OUTPUT_TEST_PINS: (no value), pie:1X03
- added ADC_INPUTS, MUX_INPUTS: (no value), pie:1X02
- added ADC_ON, AMP_ON: GREEN, pie:LED-0603
- added OUTPUT: (no value), pie:1X03
- added U$7: (no value), pie:PIE-LOGO-SMALL
- moved BATTERY_CONNECT 62.2 mm to (22.6, 5.08)
- moved EXTERNAL_POWER 55.9 mm to (36.1, 4.32)
- moved R6 48.4 mm to (18.3, 36.8)
- moved R5 41.7 mm to (18.3, 33.0)
- moved IC1 39.9 mm to (61.5, 34.3)
- moved U$2 37.5 mm to (19.6, 22.1)
- moved U$1 37.2 mm to (6.60, 11.9)
- moved U$5 32.2 mm to (6.60, 35.3)
- moved U$3 32.0 mm to (17.3, 42.2)
- moved R2 28.4 mm to (27.9, 20.6)
- moved R1 28.4 mm to (27.9, 22.6)
- moved R4 20.5 mm to (27.9, 24.6)
- moved R3 20.5 mm to (27.9, 26.7)
- moved R8 16.1 mm to (49.5, 43.9), turned to 180 degrees
- moved R7 12.8 mm to (49.0, 38.6)
Connections:
- net 1-COM: now also MUX_INPUTS.2; no longer AMP_MUX_INPUTS.2
- net 2-COM: now also MUX_INPUTS.1; no longer AMP_MUX_INPUTS.1
- net ADC_1-COM: now also ADC_INPUTS.2; no longer ADC_MUX_INPUTS.2
- net ADC_2-COM: now also ADC_INPUTS.1; no longer ADC_MUX_INPUTS.1
- net ADC_OUT: now also OUTPUT.3; no longer OUTPUT_TEST_PINS.3
- net AMP_OUT: now also OUTPUT.2; no longer OUTPUT_TEST_PINS.2
- net GND: now also OUTPUT.1; no longer OUTPUT_TEST_PINS.1
- net LED_1: now also AMP_ON.A; no longer LED1.A
- net LED_2: now also ADC_ON.A; no longer LED2.A
- net N$7: now also ADC_ON.C; no longer LED2.C
- net N$8: now also AMP_ON.C; no longer LED1.C
Routing:
- net GND: track 0.00 -> 116.5 mm, vias 0 -> 1
- net VCC: track 33.2 -> 100.5 mm
- net 2-COM: track 5.01 -> 64.6 mm, vias 0 -> 2
- net A: track 0.00 -> 55.8 mm
- net B: track 0.00 -> 52.3 mm
- net BCELL3: track 18.1 -> 64.9 mm
- net SDA: track 21.2 -> 63.6 mm
- net ADC_2-COM: track 0.00 -> 42.0 mm
- net 5V: track 48.3 -> 10.8 mm
- net ADC_A: track 72.0 -> 37.8 mm, vias 0 -> 1
- net N$3: track 47.4 -> 14.1 mm
- net SCL: track 22.4 -> 54.3 mm
- net N$2: track 43.3 -> 13.8 mm
- net ADC_OUT: track 0.00 -> 29.4 mm
- net LED_2: track 0.00 -> 27.0 mm
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Other:
- board size 81.3 x 54.6 mm -> 63.5 x 47 mm
- board text added: "(c) Pioneers In Engineering Design by: Nick W, Jehan Y This design is open source hardware. For more information, visit: https://github.com/pioneers/PiElectrical"
- board text added: "ADC 1-COM"
- board text added: "ADC 2-COM"
- board text added: "ADC_OUT"
- board text added: "ALL 10K"
- board text added: "AMP 1-COM"
- board text added: "AMP 2-COM"
- board text added: "AMP OUT"
- board text added: "EXTERNAL 5V"
- board text added: "GND"
- board text added: "PIONEERS IN ENGINEERING BATTERY BUZZER SOLUTION TEST BOARD REV 10A"

Commit message: SWAG
Parts:
- flipped U$7 to the bottom
Changed lines of the file:
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@@
 <attribute name="VALUE" x="5.969" y="19.431" size="1.27" layer="27" ratio="10" rot="R270"/>
 </element>
-<element name="U$2" library="pie" package="DIL08" value="TL072" x="19.558" y="22.098" rot="R270"/>
+<element name="U$2" library="pie" package="DIL08" value="TL072" x="19.558" y="22.098" smashed="yes" rot="R270">
+<attribute name="VALUE" x="18.923" y="25.654" size="1.27" layer="27" ratio="10" rot="R270"/>
+</element>
 <element name="U$3" library="pie" package="SOT-23_6PIN" value="SOT-23_6PIN" x="17.272" y="42.164" rot="R270"/>
 <element name="BATTERY_CONNECT" library="pie" package="XH_CONNECTOR_4POS_2.5MM" value="XH_CONNECTOR_4POS" x="22.606" y="5.08" smashed="yes">
@@
 <attribute name="VALUE" x="28.956" y="47.117" size="1.27" layer="27" font="vector" rot="R180"/>
 </element>
-<element name="U$7" library="pie" package="PIE-LOGO-SMALL" value="" x="30.734" y="21.336"/>
+<element name="U$7" library="pie" package="PIE-LOGO-SMALL" value="" x="30.734" y="21.336" rot="MR0"/>
 </elements>
 <signals>
