File: Boards/PDB/PDB.sch (EAGLE design)
At the start: 55 parts, among them Q1 NMOS, Q2 IRFML8244, Q3 PMOS, Q4 PMOS, Q5 PMOS

Commit message: I don't know
Parts:
- removed FUSE1, FUSE10, FUSE2, FUSE3, FUSE4, FUSE5, FUSE6, FUSE7, FUSE8, FUSE9: FUSE_HOLDER_SMD, pie:FUSE_HOLDER_SMD
Connections:
- removed net VOUT1: CONN1.VCC, FUSE1.1
- removed net VOUT10: CONN10.P$1, FUSE10.1
- removed net VOUT2: CONN2.VCC, FUSE2.1
- removed net VOUT3: CONN3.VCC, FUSE3.1
- removed net VOUT4: CONN4.VCC, FUSE4.2
- removed net VOUT5: CONN5.VCC, FUSE5.2
- removed net VOUT6: CONN6.VCC, FUSE6.2
- removed net VOUT7: CONN7.P$1, FUSE7.2
- removed net VOUT8: CONN9.P$1, FUSE8.1
- removed net VOUT9: CONN8.P$1, FUSE9.2
- net 12V: now also CONN1.VCC, CONN2.VCC, CONN3.VCC, CONN4.VCC, CONN5.VCC, CONN6.VCC; no longer FUSE1.2, FUSE2.2, FUSE3.2, FUSE4.1, FUSE5.1, FUSE6.1
- net 5V: now also CONN10.P$1, CONN7.P$1, CONN8.P$1, CONN9.P$1; no longer FUSE10.2, FUSE7.1, FUSE8.2, FUSE9.1
Changed lines of the file:
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@@
 <?xml version="1.0" encoding="utf-8"?>
 <!DOCTYPE eagle SYSTEM "eagle.dtd">
-<eagle version="6.6.0">
+<eagle version="8.0.0">
 <drawing>
 <settings>
@@
 <part name="CONN5" library="pie" deviceset="ANDERSON" device="VERTICAL" value="ANDERSONVERTICAL"/>
 <part name="CIRCUIT_BREAKER" library="pie" deviceset="CIRC_BREAKER" device=""/>
-<part name="FUSE4" library="pie" deviceset="FUSE_HOLDER_SMD" device=""/>
-<part name="FUSE1" library="pie" deviceset="FUSE_HOLDER_SMD" device=""/>
-<part name="FUSE2" library="pie" deviceset="FUSE_HOLDER_SMD" device=""/>
-<part name="FUSE5" library="pie" deviceset="FUSE_HOLDER_SMD" device=""/>
-<part name="FUSE3" library="pie" deviceset="FUSE_HOLDER_SMD" device=""/>
-<part name="FUSE6" library="pie" deviceset="FUSE_HOLDER_SMD" device=""/>
 <part name="CONN3" library="pie" deviceset="ANDERSON" device="VERTICAL" value="ANDERSONVERTICAL"/>
 <part name="CONN6" library="pie" deviceset="ANDERSON" device="VERTICAL" value="ANDERSONVERTICAL"/>
@@
 <part name="SUPPLY7" library="pie" deviceset="GND" device=""/>
 <part name="U$7" library="pie" deviceset="BUCK_CONVERTER_5V" device=""/>
-<part name="FUSE7" library="pie" deviceset="FUSE_HOLDER_SMD" device=""/>
-<part name="FUSE8" library="pie" deviceset="FUSE_HOLDER_SMD" device=""/>
-<part name="FUSE9" library="pie" deviceset="FUSE_HOLDER_SMD" device=""/>
-<part name="FUSE10" library="pie" deviceset="FUSE_HOLDER_SMD" device=""/>
 <part name="SUPPLY8" library="pie" deviceset="GND" device=""/>
 <part name="SUPPLY9" library="pie" deviceset="GND" device=""/>
@@
 <instance part="CONN5" gate="G$1" x="119.38" y="111.76" rot="MR0"/>
 <instance part="CIRCUIT_BREAKER" gate="G$1" x="35.56" y="132.08"/>
-<instance part="FUSE4" gate="G$1" x="101.6" y="137.16"/>
-<instance part="FUSE1" gate="G$1" x="91.44" y="147.32"/>
-<instance part="FUSE2" gate="G$1" x="91.44" y="124.46"/>
-<instance part="FUSE5" gate="G$1" x="101.6" y="114.3"/>
-<instance part="FUSE3" gate="G$1" x="91.44" y="104.14"/>
-<instance part="FUSE6" gate="G$1" x="101.6" y="96.52"/>
 <instance part="CONN3" gate="G$1" x="73.66" y="101.6"/>
 <instance part="CONN6" gate="G$1" x="119.38" y="93.98" rot="MR0"/>
@@
 <instance part="SUPPLY7" gate="GND" x="104.14" y="88.9"/>
 <instance part="U$7" gate="G$1" x="162.56" y="144.78"/>
-<instance part="FUSE7" gate="G$1" x="177.8" y="124.46" rot="MR0"/>
-<instance part="FUSE8" gate="G$1" x="187.96" y="116.84" rot="MR0"/>
-<instance part="FUSE9" gate="G$1" x="177.8" y="104.14" rot="MR0"/>
-<instance part="FUSE10" gate="G$1" x="187.96" y="93.98" rot="MR0"/>
 <instance part="SUPPLY8" gate="GND" x="193.04" y="83.82" rot="MR0"/>
 <instance part="SUPPLY9" gate="GND" x="193.04" y="106.68" rot="MR0"/>
@@
 <net name="12V" class="0">
 <segment>
-<pinref part="FUSE1" gate="G$1" pin="2"/>
-<wire x1="96.52" y1="137.16" x2="96.52" y2="124.46" width="0.1524" layer="91"/>
-<junction x="96.52" y="137.16"/>
-<pinref part="FUSE4" gate="G$1" pin="1"/>
-<pinref part="FUSE5" gate="G$1" pin="1"/>
-<junction x="96.52" y="114.3"/>
-<wire x1="96.52" y1="124.46" x2="96.52" y2="114.3" width="0.1524" layer="91"/>
-<wire x1="96.52" y1="137.16" x2="96.52" y2="147.32" width="0.1524" layer="91"/>
-<wire x1="96.52" y1="114.3" x2="96.52" y2="104.14" width="0.1524" layer="91"/>
-<wire x1="96.52" y1="104.14" x2="96.52" y2="96.52" width="0.1524" layer="91"/>
-<pinref part="FUSE3" gate="G$1" pin="2"/>
-<junction x="96.52" y="104.14"/>
-<pinref part="FUSE6" gate="G$1" pin="1"/>
-<pinref part="FUSE2" gate="G$1" pin="2"/>
-<junction x="96.52" y="124.46"/>
-<wire x1="96.52" y1="147.32" x2="109.22" y2="147.32" width="0.1524" layer="91"/>
-<label x="101.6" y="147.32" size="1.778" layer="95"/>
-</segment>
-<segment>
 <pinref part="CIRCUIT_BREAKER" gate="G$1" pin="P$2"/>
 <wire x1="35.56" y1="119.38" x2="35.56" y2="116.84" width="0.1524" layer="91"/>
@@
 <label x="142.24" y="147.32" size="1.778" layer="95"/>
 </segment>
-</net>
-<net name="VOUT1" class="0">
-<segment>
+<segment>
+<pinref part="CONN6" gate="G$1" pin="VCC"/>
+<pinref part="CONN3" gate="G$1" pin="VCC"/>
+<pinref part="CONN5" gate="G$1" pin="VCC"/>
+<pinref part="CONN4" gate="G$1" pin="VCC"/>
+<pinref part="CONN2" gate="G$1" pin="VCC"/>
+<wire x1="96.52" y1="147.32" x2="96.52" y2="137.16" width="0.1524" layer="91"/>
+<wire x1="96.52" y1="137.16" x2="96.52" y2="124.46" width="0.1524" layer="91"/>
+<wire x1="96.52" y1="124.46" x2="96.52" y2="114.3" width="0.1524" layer="91"/>
+<wire x1="96.52" y1="114.3" x2="96.52" y2="104.14" width="0.1524" layer="91"/>
+<wire x1="96.52" y1="104.14" x2="96.52" y2="96.52" width="0.1524" layer="91"/>
+<wire x1="96.52" y1="147.32" x2="109.22" y2="147.32" width="0.1524" layer="91"/>
+<label x="101.6" y="147.32" size="1.778" layer="95"/>
 <pinref part="CONN1" gate="G$1" pin="VCC"/>
-<wire x1="86.36" y1="147.32" x2="81.28" y2="147.32" width="0.1524" layer="91"/>
-<pinref part="FUSE1" gate="G$1" pin="1"/>
-</segment>
-</net>
-<net name="VOUT2" class="0">
-<segment>
-<pinref part="CONN2" gate="G$1" pin="VCC"/>
-<wire x1="86.36" y1="124.46" x2="81.28" y2="124.46" width="0.1524" layer="91"/>
-<pinref part="FUSE2" gate="G$1" pin="1"/>
-</segment>
-</net>
-<net name="VOUT4" class="0">
-<segment>
-<pinref part="CONN4" gate="G$1" pin="VCC"/>
-<wire x1="111.76" y1="137.16" x2="106.68" y2="137.16" width="0.1524" layer="91"/>
-<pinref part="FUSE4" gate="G$1" pin="2"/>
-</segment>
-</net>
-<net name="VOUT5" class="0">
-<segment>
-<pinref part="FUSE5" gate="G$1" pin="2"/>
-<pinref part="CONN5" gate="G$1" pin="VCC"/>
-<wire x1="106.68" y1="114.3" x2="111.76" y2="114.3" width="0.1524" layer="91"/>
-</segment>
-</net>
-<net name="VOUT3" class="0">
-<segment>
-<pinref part="FUSE3" gate="G$1" pin="1"/>
-<pinref part="CONN3" gate="G$1" pin="VCC"/>
-<wire x1="86.36" y1="104.14" x2="81.28" y2="104.14" width="0.1524" layer="91"/>
+<wire x1="96.52" y1="147.32" x2="81.28" y2="147.32" width="0.1524" layer="91"/>
+<junction x="96.52" y="147.32"/>
+<wire x1="81.28" y1="124.46" x2="96.52" y2="124.46" width="0.1524" layer="91"/>
+<junction x="96.52" y="124.46"/>
+<wire x1="111.76" y1="137.16" x2="96.52" y2="137.16" width="0.1524" layer="91"/>
+<junction x="96.52" y="137.16"/>
+<wire x1="111.76" y1="114.3" x2="96.52" y2="114.3" width="0.1524" layer="91"/>
+<junction x="96.52" y="114.3"/>
+<wire x1="81.28" y1="104.14" x2="96.52" y2="104.14" width="0.1524" layer="91"/>
+<junction x="96.52" y="104.14"/>
+<wire x1="111.76" y1="96.52" x2="96.52" y2="96.52" width="0.1524" layer="91"/>
 </segment>
 </net>
@@
 </segment>
 </net>
-<net name="VOUT6" class="0">
-<segment>
-<pinref part="FUSE6" gate="G$1" pin="2"/>
-<wire x1="106.68" y1="96.52" x2="111.76" y2="96.52" width="0.1524" layer="91"/>
-<pinref part="CONN6" gate="G$1" pin="VCC"/>
-</segment>
-</net>
-<net name="VOUT7" class="0">
-<segment>
-<pinref part="FUSE7" gate="G$1" pin="2"/>
-<wire x1="172.72" y1="124.46" x2="160.02" y2="124.46" width="0.1524" layer="91"/>
+<net name="5V" class="0">
+<segment>
+<pinref part="CONN10" gate="CONN$1" pin="P$1"/>
+<pinref part="CONN8" gate="CONN$1" pin="P$1"/>
+<pinref part="CONN9" gate="CONN$1" pin="P$1"/>
 <pinref part="CONN7" gate="CONN$1" pin="P$1"/>
-</segment>
-</net>
-<net name="VOUT8" class="0">
-<segment>
-<pinref part="FUSE8" gate="G$1" pin="1"/>
-<wire x1="193.04" y1="116.84" x2="198.12" y2="116.84" width="0.1524" layer="91"/>
-<pinref part="CONN9" gate="CONN$1" pin="P$1"/>
-</segment>
-</net>
-<net name="VOUT9" class="0">
-<segment>
-<pinref part="FUSE9" gate="G$1" pin="2"/>
-<wire x1="172.72" y1="104.14" x2="162.56" y2="104.14" width="0.1524" layer="91"/>
-<pinref part="CONN8" gate="CONN$1" pin="P$1"/>
-</segment>
-</net>
-<net name="VOUT10" class="0">
-<segment>
-<pinref part="FUSE10" gate="G$1" pin="1"/>
-<wire x1="193.04" y1="93.98" x2="198.12" y2="93.98" width="0.1524" layer="91"/>
-<pinref part="CONN10" gate="CONN$1" pin="P$1"/>
-</segment>
-</net>
-<net name="5V" class="0">
-<segment>
+<wire x1="182.88" y1="124.46" x2="160.02" y2="124.46" width="0.1524" layer="91"/>
 <pinref part="U$7" gate="G$1" pin="OUT+"/>
 <wire x1="175.26" y1="147.32" x2="182.88" y2="147.32" width="0.1524" layer="91"/>
 <wire x1="182.88" y1="147.32" x2="182.88" y2="124.46" width="0.1524" layer="91"/>
-<pinref part="FUSE10" gate="G$1" pin="2"/>
+<label x="180.34" y="147.32" size="1.778" layer="95" ratio="10"/>
 <wire x1="182.88" y1="124.46" x2="182.88" y2="116.84" width="0.1524" layer="91"/>
+<junction x="182.88" y="124.46"/>
 <wire x1="182.88" y1="116.84" x2="182.88" y2="104.14" width="0.1524" layer="91"/>
 <wire x1="182.88" y1="104.14" x2="182.88" y2="93.98" width="0.1524" layer="91"/>
-<pinref part="FUSE9" gate="G$1" pin="1"/>
-<pinref part="FUSE8" gate="G$1" pin="2"/>
-<pinref part="FUSE7" gate="G$1" pin="1"/>
-<junction x="182.88" y="124.46"/>
+<wire x1="198.12" y1="116.84" x2="182.88" y2="116.84" width="0.1524" layer="91"/>
 <junction x="182.88" y="116.84"/>
+<wire x1="162.56" y1="104.14" x2="182.88" y2="104.14" width="0.1524" layer="91"/>
 <junction x="182.88" y="104.14"/>
-<label x="180.34" y="147.32" size="1.778" layer="95" ratio="10"/>
+<wire x1="198.12" y1="93.98" x2="182.88" y2="93.98" width="0.1524" layer="91"/>
 </segment>
 </net>

Commit message: REV B PLEASE WORK
Parts:
- removed U$7: BUCK_CONVERTER_5V, pie:BUCK_CONVERTER_5V
Connections:
- net 12V: no longer U$7.IN+
- net 5V: no longer U$7.OUT+
- net GND: no longer U$7.IN-, U$7.OUT-
Changed lines of the file:
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@@
 <part name="SUPPLY6" library="pie" deviceset="GND" device=""/>
 <part name="SUPPLY7" library="pie" deviceset="GND" device=""/>
-<part name="U$7" library="pie" deviceset="BUCK_CONVERTER_5V" device=""/>
 <part name="SUPPLY8" library="pie" deviceset="GND" device=""/>
 <part name="SUPPLY9" library="pie" deviceset="GND" device=""/>
@@
 <instance part="SUPPLY6" gate="GND" x="83.82" y="96.52"/>
 <instance part="SUPPLY7" gate="GND" x="104.14" y="88.9"/>
-<instance part="U$7" gate="G$1" x="162.56" y="144.78"/>
 <instance part="SUPPLY8" gate="GND" x="193.04" y="83.82" rot="MR0"/>
 <instance part="SUPPLY9" gate="GND" x="193.04" y="106.68" rot="MR0"/>
@@
 </segment>
 <segment>
-<pinref part="U$7" gate="G$1" pin="IN+"/>
 <wire x1="149.86" y1="147.32" x2="142.24" y2="147.32" width="0.1524" layer="91"/>
 <label x="142.24" y="147.32" size="1.778" layer="95"/>
@@
 </segment>
 <segment>
-<pinref part="U$7" gate="G$1" pin="IN-"/>
 <wire x1="149.86" y1="142.24" x2="139.7" y2="142.24" width="0.1524" layer="91"/>
 <pinref part="SUPPLY12" gate="GND" pin="GND"/>
 </segment>
 <segment>
-<pinref part="U$7" gate="G$1" pin="OUT-"/>
 <pinref part="SUPPLY13" gate="GND" pin="GND"/>
 <wire x1="175.26" y1="142.24" x2="177.8" y2="142.24" width="0.1524" layer="91"/>
@@
 <pinref part="CONN7" gate="CONN$1" pin="P$1"/>
 <wire x1="182.88" y1="124.46" x2="160.02" y2="124.46" width="0.1524" layer="91"/>
-<pinref part="U$7" gate="G$1" pin="OUT+"/>
 <wire x1="175.26" y1="147.32" x2="182.88" y2="147.32" width="0.1524" layer="91"/>
 <wire x1="182.88" y1="147.32" x2="182.88" y2="124.46" width="0.1524" layer="91"/>
