File: Boards/MotorController/MCChipProto.sch (EAGLE design)
At the start: 7 parts, among them IC1 MC33926

Commit message: Finished prototype board
Parts:
- removed U$1: 2X5PIN, pie:2X5PIN
- added J1: MC BREAKOUT, pie:2X5PIN
Connections:
- net 3.3V: now also J1.3.3V; no longer U$1.3.3V
- net ADC: now also J1.ADC; no longer U$1.ADC
- net GND: now also J1.GND; no longer U$1.GND
- net IN1: now also J1.IN1; no longer U$1.IN1
- net IN2: now also J1.IN2; no longer U$1.IN2
- net INV: now also J1.INV; no longer U$1.INV
- net OUT1: now also J1.OUT1; no longer U$1.OUT1
- net OUT2: now also J1.OUT2; no longer U$1.OUT2
- net SLEW: now also J1.SLEW; no longer U$1.SLEW
- net VCC: now also J1.VCC; no longer U$1.VCC
Other:
- moved on the sheet: C1, C2, C3, C4, IC1, R1
