File: Boards/MotorController/MotorController.sch (EAGLE design)
At the start: 15 parts, among them IC1 MC33926

Commit message: Modifying motor controller
Connections:
- removed net PWM: APM.9, IC1.IN1
- new net PWM1: APM.8, IC1.IN1
- new net PWM2: APM.9, IC1.IN2
- net GND: no longer IC1.IN2
- net INV: now also APM.7; no longer APM.8
Changed lines of the file:
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@@
 <part name="C4" library="pie" deviceset="CAP_POL" device="RADIAL" value="100 uF"/>
 <part name="R3" library="pie" deviceset="R-US_" device="R0603" value="200"/>
-<part name="SUPPLY13" library="pie" deviceset="GND" device=""/>
 <part name="CONN1" library="pie" deviceset="ANDERSON" device="VERTICAL"/>
 <part name="CONN2" library="pie" deviceset="ANDERSON" device="VERTICAL"/>
@@
 <instance part="C4" gate="G$1" x="167.64" y="142.24" rot="R270"/>
 <instance part="R3" gate="G$1" x="137.16" y="68.58" rot="R90"/>
-<instance part="SUPPLY13" gate="GND" x="152.4" y="106.68"/>
 <instance part="CONN1" gate="G$1" x="154.94" y="167.64"/>
 <instance part="CONN2" gate="G$1" x="195.58" y="167.64"/>
@@
 </segment>
 <segment>
-<pinref part="IC1" gate="G$1" pin="IN2"/>
-<wire x1="157.48" y1="109.22" x2="152.4" y2="109.22" width="0.1524" layer="91"/>
-<pinref part="SUPPLY13" gate="GND" pin="GND"/>
-</segment>
-<segment>
 <pinref part="CONN2" gate="G$1" pin="OUTB"/>
 <wire x1="203.2" y1="165.1" x2="205.74" y2="165.1" width="0.1524" layer="91"/>
@@
 <wire x1="76.2" y1="78.74" x2="78.74" y2="78.74" width="0.1524" layer="91"/>
 <label x="78.74" y="78.74" size="1.778" layer="95"/>
-</segment>
-</net>
-<net name="PWM" class="0">
-<segment>
-<pinref part="APM" gate="APM" pin="9"/>
-<wire x1="48.26" y1="78.74" x2="45.72" y2="78.74" width="0.1524" layer="91"/>
-<label x="43.18" y="78.74" size="1.778" layer="95"/>
-</segment>
-<segment>
-<pinref part="IC1" gate="G$1" pin="IN1"/>
-<wire x1="157.48" y1="99.06" x2="152.4" y2="99.06" width="0.1524" layer="91"/>
-<label x="149.86" y="99.06" size="1.778" layer="95"/>
 </segment>
 </net>
@@
 <net name="INV" class="0">
 <segment>
+<pinref part="IC1" gate="G$1" pin="INV"/>
+<wire x1="157.48" y1="86.36" x2="152.4" y2="86.36" width="0.1524" layer="91"/>
+<label x="149.86" y="86.36" size="1.778" layer="95"/>
+</segment>
+<segment>
+<pinref part="APM" gate="APM" pin="7"/>
+<wire x1="48.26" y1="83.82" x2="45.72" y2="83.82" width="0.1524" layer="91"/>
+<label x="43.18" y="83.82" size="1.778" layer="95"/>
+</segment>
+</net>
+<net name="PWM1" class="0">
+<segment>
 <pinref part="APM" gate="APM" pin="8"/>
 <wire x1="48.26" y1="81.28" x2="45.72" y2="81.28" width="0.1524" layer="91"/>
@@
 </segment>
 <segment>
-<pinref part="IC1" gate="G$1" pin="INV"/>
-<wire x1="157.48" y1="86.36" x2="152.4" y2="86.36" width="0.1524" layer="91"/>
-<label x="149.86" y="86.36" size="1.778" layer="95"/>
-</segment>
-</net>
+<pinref part="IC1" gate="G$1" pin="IN1"/>
+<wire x1="157.48" y1="99.06" x2="152.4" y2="99.06" width="0.1524" layer="91"/>
+<label x="149.86" y="99.06" size="1.778" layer="95"/>
+</segment>
+</net>
+<net name="PWM2" class="0">
+<segment>
+<pinref part="APM" gate="APM" pin="9"/>
+<wire x1="48.26" y1="78.74" x2="45.72" y2="78.74" width="0.1524" layer="91"/>
+<label x="43.18" y="78.74" size="1.778" layer="95"/>
+</segment>
+<segment>
+<pinref part="IC1" gate="G$1" pin="IN2"/>
+<wire x1="157.48" y1="109.22" x2="152.4" y2="109.22" width="0.1524" layer="91"/>
+<label x="149.86" y="109.22" size="1.778" layer="95"/>
+</segment>
+</net>

Commit message: Rev B Motor Controller
Parts:
- added U$7: 5PIN5PIN_MC, pie:5PIN5PIN_MC
Connections:
- net GND: now also CONN2.OUTA, U$7.GND; no longer CONN2.OUTB
- net INV: now also U$7.P1
- net OUT1: now also CONN1.OUTB; no longer CONN1.OUTA
- net OUT2: now also CONN1.OUTA; no longer CONN1.OUTB
- net PWM1: now also U$7.P2
- net PWM2: now also U$7.P3
- net VCC: now also U$7.VCC
- net VPWR: now also CONN2.OUTB; no longer CONN2.OUTA
Changed lines of the file:
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@@
 <part name="FRAME1" library="pie" deviceset="FRAME_SCHEMATIC" device="">
 <attribute name="AUTHOR" value="Seiya O, Averal K, Margo O, Steven L"/>
-<attribute name="REVISION" value="A"/>
+<attribute name="REVISION" value="B"/>
 </part>
 <part name="SUPPLY2" library="pie" deviceset="GND" device=""/>
@@
 <part name="CONN2" library="pie" deviceset="ANDERSON" device="VERTICAL"/>
 <part name="SUPPLY14" library="pie" deviceset="GND" device=""/>
+<part name="U$7" library="pie" deviceset="5PIN" device="5PIN_MC"/>
+<part name="SUPPLY13" library="pie" deviceset="GND" device=""/>
 </parts>
 <sheets>
@@
 <instance part="CONN1" gate="G$1" x="154.94" y="167.64"/>
 <instance part="CONN2" gate="G$1" x="195.58" y="167.64"/>
-<instance part="SUPPLY14" gate="GND" x="210.82" y="160.02"/>
+<instance part="SUPPLY14" gate="GND" x="220.98" y="165.1"/>
+<instance part="U$7" gate="G$1" x="91.44" y="114.3"/>
+<instance part="SUPPLY13" gate="GND" x="99.06" y="101.6"/>
 </instances>
 <busses>
@@
 </segment>
 <segment>
-<pinref part="CONN2" gate="G$1" pin="OUTB"/>
-<wire x1="203.2" y1="165.1" x2="205.74" y2="165.1" width="0.1524" layer="91"/>
+<pinref part="U$7" gate="G$1" pin="GND"/>
+<wire x1="99.06" y1="109.22" x2="99.06" y2="104.14" width="0.1524" layer="91"/>
+<pinref part="SUPPLY13" gate="GND" pin="GND"/>
+</segment>
+<segment>
+<pinref part="CONN2" gate="G$1" pin="OUTA"/>
+<wire x1="203.2" y1="170.18" x2="220.98" y2="170.18" width="0.1524" layer="91"/>
 <pinref part="SUPPLY14" gate="GND" pin="GND"/>
-<wire x1="205.74" y1="165.1" x2="210.82" y2="165.1" width="0.1524" layer="91"/>
-<wire x1="210.82" y1="165.1" x2="210.82" y2="162.56" width="0.1524" layer="91"/>
+<wire x1="220.98" y1="170.18" x2="220.98" y2="167.64" width="0.1524" layer="91"/>
 </segment>
 </net>
@@
 <wire x1="76.2" y1="99.06" x2="78.74" y2="99.06" width="0.1524" layer="91"/>
 <label x="78.74" y="99.06" size="1.778" layer="95"/>
+</segment>
+<segment>
+<pinref part="U$7" gate="G$1" pin="VCC"/>
+<wire x1="129.54" y1="109.22" x2="129.54" y2="104.14" width="0.1524" layer="91"/>
+<label x="127" y="101.6" size="1.778" layer="95"/>
 </segment>
 </net>
@@
 </segment>
 <segment>
-<pinref part="CONN1" gate="G$1" pin="OUTA"/>
-<wire x1="162.56" y1="170.18" x2="165.1" y2="170.18" width="0.1524" layer="91"/>
-<label x="165.1" y="170.18" size="1.778" layer="95"/>
+<pinref part="CONN1" gate="G$1" pin="OUTB"/>
+<wire x1="162.56" y1="165.1" x2="165.1" y2="165.1" width="0.1524" layer="91"/>
+<label x="165.1" y="165.1" size="1.778" layer="95"/>
 </segment>
 </net>
@@
 </segment>
 <segment>
-<pinref part="CONN1" gate="G$1" pin="OUTB"/>
-<wire x1="162.56" y1="165.1" x2="165.1" y2="165.1" width="0.1524" layer="91"/>
-<label x="165.1" y="165.1" size="1.778" layer="95"/>
+<pinref part="CONN1" gate="G$1" pin="OUTA"/>
+<wire x1="162.56" y1="170.18" x2="165.1" y2="170.18" width="0.1524" layer="91"/>
+<label x="165.1" y="170.18" size="1.778" layer="95"/>
 </segment>
 </net>
@@
 </segment>
 <segment>
-<pinref part="CONN2" gate="G$1" pin="OUTA"/>
-<wire x1="203.2" y1="170.18" x2="205.74" y2="170.18" width="0.1524" layer="91"/>
-<label x="205.74" y="170.18" size="1.778" layer="95"/>
+<pinref part="CONN2" gate="G$1" pin="OUTB"/>
+<wire x1="203.2" y1="165.1" x2="205.74" y2="165.1" width="0.1524" layer="91"/>
+<label x="205.74" y="165.1" size="1.778" layer="95"/>
 </segment>
 </net>
@@
 <label x="43.18" y="83.82" size="1.778" layer="95"/>
 </segment>
+<segment>
+<pinref part="U$7" gate="G$1" pin="P1"/>
+<wire x1="121.92" y1="109.22" x2="121.92" y2="104.14" width="0.1524" layer="91"/>
+<label x="119.38" y="101.6" size="1.778" layer="95"/>
+</segment>
 </net>
 <net name="PWM1" class="0">
@@
 <label x="149.86" y="99.06" size="1.778" layer="95"/>
 </segment>
+<segment>
+<pinref part="U$7" gate="G$1" pin="P2"/>
+<wire x1="114.3" y1="109.22" x2="114.3" y2="104.14" width="0.1524" layer="91"/>
+<label x="111.76" y="101.6" size="1.778" layer="95"/>
+</segment>
 </net>
 <net name="PWM2" class="0">
@@
 <label x="149.86" y="109.22" size="1.778" layer="95"/>
 </segment>
-</net>
+<segment>
+<pinref part="U$7" gate="G$1" pin="P3"/>
+<wire x1="106.68" y1="109.22" x2="106.68" y2="104.14" width="0.1524" layer="91"/>
+<label x="104.14" y="101.6" size="1.778" layer="95"/>
+</segment>
+</net>
