File: Boards/PDB2/PDB/PDB2.brd (EAGLE design)
At the start: 102.6 x 71.8 mm, 51 parts, among them J1 XT60CONNECTOR, J10 AVR_SPI_PROG_5X2LOCK, J3 ANDERSONVERTICAL, J4 ANDERSONVERTICAL, J5 ATX, J6 ATX, J7 ATX, J8 ATX, M1 STD20NF06LDPAK-M, M2 STD20NF06LDPAK-M, U1 BQ7692006PWRPW20-M, U2 Value

Commit message: yeet
Parts:
- removed R4: 100, pie:R0603
- added J12: (no value), SparkFun-Connectors:1X02
- added R20: 100k, pie:R0603
- C5, C8: device pie:0603-CAP -> pie:0805
- R6: value 10k -> 5.6k
- R8: value 3m -> 5m; device pie:R2512 -> pie:SMD_SHUNT
- Y1: device pie:HC49UP -> pie:SMD_CRYSTAL
- moved C9 4.70 mm to (93.9, 19.8)
- moved C10 4.59 mm to (93.6, 30.7)
- moved Y1 1.14 mm to (93.9, 25.1), turned to 270 degrees
- moved C4 0.85 mm to (63.1, 16.5)
- moved R6 0.74 mm to (69.3, 32.6), turned to 270 degrees
- moved R8 0.40 mm to (31.4, 15.7)
- moved C5 0.25 mm to (31.6, 37.7)
- moved C8 0.18 mm to (53.3, 38.0)
Connections:
- removed net N$3: D1.2, R4.2, R5.1
- new net PG: R20.1, U2.4, U3.26
- new net RXD: J12.1, U3.30
- new net TXD: J12.2, U3.31
- net 5V: now also R20.2, U2.14, U2.7
- net DSG: now also R6.2; no longer R6.1
- net GND: now also R6.1, R8.P$1, Y1.P1, Y1.P3; no longer R6.2, R8.1
- net GND_OUT: no longer U2.7
- net N$4: no longer U2.14
- net N$5: now also Y1.P2; no longer Y1.1
- net N$7: now also Y1.P0; no longer Y1.2
- net SRP: now also R8.P$2; no longer R8.2
- net VIN: now also D1.2, R5.1; no longer R4.1
Routing:
- net PG: track 0.00 -> 45.6 mm, vias 0 -> 2
- net GND: track 0.00 -> 43.6 mm, vias 65 -> 68
- net 5V: track 0.00 -> 28.4 mm, vias 0 -> 2
- net TXD: track 0.00 -> 18.3 mm, vias 0 -> 1
- net RXD: track 0.00 -> 15.2 mm, vias 0 -> 1
- net SRP: track 24.9 -> 34.6 mm
- net VIN: track 8.15 -> 15.1 mm
- net N$3: track 5.93 -> 0.00 mm
- net N$5: track 20.2 -> 15.2 mm
- net N$4: track 3.88 -> 0.00 mm
- net N$7: track 13.0 -> 11.6 mm
- net GND_OUT: track 9.33 -> 8.18 mm, vias 75 -> 79
- net BCELL1: track 42.3 -> 42.8 mm, vias 1 -> 0
- net BCELL3: track 25.0 -> 25.3 mm, vias 1 -> 0
- net BCELL2: track 25.1 -> 25.2 mm, vias 1 -> 0
Other:
- board text added: "ON/OFF"
- board text added: "RXD"
- board text added: "TXD"
