File: Boards/PDB2/PDB/PDB2_1.brd (EAGLE design)
At the start: 112.1 x 89.9 mm, 76 parts, among them J1 XT60CONNECTOR, J2 AVR_SPI_PRG_6MA03-2, J3 USB_B_PTH, M1 STD20NF06LDPAK-M, M2 STD20NF06LDPAK-M, SW1 PUSH_BUTTON, U1 BQ7692006PWRPW20-M, U2 Value, U3 ATMEGA32U4-AU

Commit message: isp pls
Parts:
- added J4: AVR_SPI_PRG_6MA03-2, pie:MA03-2
Connections:
- new net MISO: J4.1
- new net N$10: J4.5
- new net N$7: J4.3
- net GND: now also J4.6
- net MOSI: now also J4.4
- net VCC: now also J4.2

Commit message: trerewrewr
Parts:
- removed J4: AVR_SPI_PRG_6MA03-2, pie:MA03-2
- removed JP6: (no value), pie:1X03-JMP-OPTION
- removed M1, M2: STD20NF06LDPAK-M, pie:DPAK-M
- removed R9: 100k, pie:R0603
- added M3: NMOS_CSD17579Q3A, pie:DNH0008A
- R6: value 5.6k -> 100k
- moved R8 16.9 mm to (44.8, 43.1), turned to 0 degrees
Connections:
- removed net MISO: J4.1
- removed net N$10: J4.5
- removed net N$26: JP6.2, R8.1
- removed net N$7: J4.3
- net 12V: now also R8.1; no longer JP6.1
- net DSG: now also M3.4; no longer M1.1, M2.1
- net EN/MISO: no longer JP6.3
- net GND: no longer C11.MINUS, C14.MINUS, C5.1, C6.1, C7.1, C9.1, J4.6, JP2.P$2, JP3.P$2, JP4.P$2, JP5.P$2, R11.1, U2.1
- net GND_OUT: now also C11.MINUS, C14.MINUS, C5.1, C6.1, C7.1, C9.1, JP2.P$2, JP3.P$2, JP4.P$2, JP5.P$2, M3.5, M3.6, M3.7, M3.8, M3.9, R11.1, U2.1; no longer M1.3, M2.3
- net MOSI: no longer J4.4
- net PG: no longer R9.1, U2.4
- net SRP: now also M3.1, M3.2, M3.3; no longer M1.2, M2.2
- net VCC: no longer J4.2, R9.2
Routing:
- net PG: track 62.2 -> 0.00 mm, vias 2 -> 0
- net EN/MISO: track 75.9 -> 30.9 mm, vias 1 -> 0
- net VCC: track 87.9 -> 53.7 mm
- net 12V: track 76.4 -> 56.6 mm
- net N$26: track 8.80 -> 0.00 mm, vias 0 -> 1
- net N$27: track 12.7 -> 4.83 mm, vias 2 -> 0
- net DSG: track 53.1 -> 46.7 mm
- net GND: vias 148 -> 106

Commit message: done with pdb rev 4
Parts:
- added C17: 2.2uF, pie:0603-CAP
- added STANDOFF1, STANDOFF2, STANDOFF3, STANDOFF4, STANDOFF5, STANDOFF7: STAND-OFFTIGHT, pie:STAND-OFF-TIGHT
- moved C12 16.7 mm to (107.6, 24.1), turned to 270 degrees
- moved Y1 16.3 mm to (107.6, 14.2)
- moved C13 16.1 mm to (109.6, 4.32), turned to 90 degrees
- moved U$1 6.74 mm to (99.8, 84.2)
- moved U$2 4.12 mm to (99.8, 79.9), flipped to the bottom
- moved LED1 0.40 mm to (99.8, 10.2)
- renumbered M3 to M1
Connections:
- net GND: now also C17.1
- net VIN: now also C17.2
Routing:
- net N$5: track 22.3 -> 38.1 mm
- net N$2: track 19.1 -> 25.0 mm
- net VIN: track 14.6 -> 18.5 mm
- net GND: vias 106 -> 104
Other:
- board text removed: "EN"
- board text removed: "uC"

Commit message: fixed lib
Parts:
- moved M1 0.13 mm to (33.8, 23.1)
Connections:
- net GND_OUT: no longer M1.6, M1.7, M1.8, M1.9
- net SRP: no longer M1.2, M1.3
