File: Boards/PDB2/PDB/PDB2_1.sch (EAGLE design)
At the start: 74 parts, among them J1 XT60CONNECTOR, J2 AVR_SPI_PRG_6MA03-2, J3 USB_B_PTH, M1 STD20NF06LDPAK-M, M2 STD20NF06LDPAK-M, SW1 PUSH_BUTTON, U1 BQ7692006PWRPW20-M, U2 Value, U3 ATMEGA32U4-AU

Commit message: trerewrewr
Parts:
- removed JP6: (no value), pie:JMP-OPTION
- removed M1, M2: STD20NF06LDPAK-M, pie:STD20NF06LDPAK-M
- removed R9: 100k, pie:R-US_R0603
- added M3: NMOS_CSD17579Q3A, pie:NMOS_CSD17579Q3A
- R6: value 5.6k -> 100k
Connections:
- removed net N$26: JP6.COMMON, R8.1
- net 12V: now also R8.1; no longer JP6.1
- net DSG: now also M3.G; no longer M1.1, M2.1
- net EN/MISO: no longer JP6.3
- net GND: no longer C11.-, C14.-, C5.1, C6.1, C7.1, C9.1, JP2.P$2, JP3.P$2, JP4.P$2, JP5.P$2, R11.1, U2.GND
- net GND_OUT: now also C11.-, C14.-, C5.1, C6.1, C7.1, C9.1, JP2.P$2, JP3.P$2, JP4.P$2, JP5.P$2, M3.D, R11.1, U2.GND; no longer M1.2, M2.2
- net PG: no longer R9.1, U2.PG
- net SRP: now also M3.S@2; no longer M1.3, M2.3
- net VCC: no longer R9.2

Commit message: done with pdb rev 4
Parts:
- added C17: 2.2uF, pie:CAP0603-CAP
- added STANDOFF1, STANDOFF2, STANDOFF3, STANDOFF4, STANDOFF5, STANDOFF7: STAND-OFFTIGHT, pie:STAND-OFFTIGHT
- renumbered M3 to M1
Connections:
- net GND: now also C17.1
- net VIN: now also C17.2
Changed lines of the file:
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@@
 <part name="C14" library="pie" deviceset="CAP_POL" device="RADIAL" value="10uF"/>
 <part name="J3" library="SparkFun-Connectors" deviceset="USB_B" device="_PTH"/>
-<part name="M3" library="pie" deviceset="NMOS_CSD17579Q3A" device=""/>
+<part name="M1" library="pie" deviceset="NMOS_CSD17579Q3A" device=""/>
+<part name="STANDOFF1" library="pie" deviceset="STAND-OFF" device="TIGHT"/>
+<part name="STANDOFF2" library="pie" deviceset="STAND-OFF" device="TIGHT"/>
+<part name="STANDOFF3" library="pie" deviceset="STAND-OFF" device="TIGHT"/>
+<part name="STANDOFF4" library="pie" deviceset="STAND-OFF" device="TIGHT"/>
+<part name="STANDOFF5" library="pie" deviceset="STAND-OFF" device="TIGHT"/>
+<part name="STANDOFF7" library="pie" deviceset="STAND-OFF" device="TIGHT"/>
+<part name="C17" library="pie" deviceset="CAP" device="0603-CAP" value="2.2uF"/>
 </parts>
 <sheets>
@@
 <attribute name="VALUE" x="-73.66" y="76.2" size="1.778" layer="96" rot="R270"/>
 </instance>
-<instance part="M3" gate="A" x="76.2" y="22.86" smashed="yes">
+<instance part="M1" gate="A" x="76.2" y="22.86" smashed="yes">
 <attribute name="NAME" x="81.28" y="22.86" size="1.778" layer="95"/>
 <attribute name="VALUE" x="81.28" y="20.32" size="1.778" layer="96"/>
+</instance>
+<instance part="STANDOFF1" gate="G$1" x="-109.22" y="86.36" smashed="yes"/>
+<instance part="STANDOFF2" gate="G$1" x="-99.06" y="86.36" smashed="yes"/>
+<instance part="STANDOFF3" gate="G$1" x="-106.68" y="76.2" smashed="yes"/>
+<instance part="STANDOFF4" gate="G$1" x="-99.06" y="78.74" smashed="yes"/>
+<instance part="STANDOFF5" gate="G$1" x="-101.6" y="68.58" smashed="yes"/>
+<instance part="STANDOFF7" gate="G$1" x="-99.06" y="60.96" smashed="yes"/>
+<instance part="C17" gate="G$1" x="-76.2" y="-17.78" smashed="yes" rot="R90">
+<attribute name="NAME" x="-78.74" y="-21.59" size="1.778" layer="95" rot="R90"/>
+<attribute name="VALUE" x="-71.12" y="-21.59" size="1.778" layer="96" rot="R90"/>
 </instance>
 </instances>
@@
 <wire x1="-114.3" y1="-5.08" x2="-106.68" y2="-5.08" width="0.1524" layer="91"/>
 <wire x1="-106.68" y1="-5.08" x2="-106.68" y2="-35.56" width="0.1524" layer="91"/>
-<wire x1="-106.68" y1="-35.56" x2="-68.58" y2="-35.56" width="0.1524" layer="91"/>
+<wire x1="-106.68" y1="-35.56" x2="-76.2" y2="-35.56" width="0.1524" layer="91"/>
+<pinref part="C17" gate="G$1" pin="1"/>
+<wire x1="-76.2" y1="-35.56" x2="-68.58" y2="-35.56" width="0.1524" layer="91"/>
+<wire x1="-76.2" y1="-20.32" x2="-76.2" y2="-35.56" width="0.1524" layer="91"/>
+<junction x="-76.2" y="-35.56"/>
 </segment>
 <segment>
@@
 <junction x="66.04" y="25.4"/>
 <pinref part="R6" gate="G$1" pin="2"/>
-<pinref part="M3" gate="A" pin="G"/>
+<pinref part="M1" gate="A" pin="G"/>
 <wire x1="68.58" y1="25.4" x2="68.58" y2="20.32" width="0.1524" layer="91"/>
 </segment>
@@
 <wire x1="-88.9" y1="0" x2="-88.9" y2="-7.62" width="0.1524" layer="91"/>
 <junction x="-88.9" y="-7.62"/>
-<wire x1="-88.9" y1="-7.62" x2="-68.58" y2="-7.62" width="0.1524" layer="91"/>
+<wire x1="-88.9" y1="-7.62" x2="-76.2" y2="-7.62" width="0.1524" layer="91"/>
 <pinref part="D2" gate="G$1" pin="C"/>
+<pinref part="C17" gate="G$1" pin="2"/>
+<wire x1="-76.2" y1="-7.62" x2="-68.58" y2="-7.62" width="0.1524" layer="91"/>
+<wire x1="-76.2" y1="-7.62" x2="-76.2" y2="-12.7" width="0.1524" layer="91"/>
+<junction x="-76.2" y="-7.62"/>
 </segment>
 </net>
@@
 <pinref part="R7" gate="G$1" pin="2"/>
 <junction x="76.2" y="7.62"/>
-<pinref part="M3" gate="A" pin="S@2"/>
+<pinref part="M1" gate="A" pin="S@2"/>
 </segment>
 </net>
@@
 <wire x1="73.66" y1="38.1" x2="76.2" y2="38.1" width="0.1524" layer="91"/>
 <label x="71.12" y="38.1" size="1.778" layer="95"/>
-<pinref part="M3" gate="A" pin="D"/>
+<pinref part="M1" gate="A" pin="D"/>
 <wire x1="73.66" y1="33.02" x2="76.2" y2="33.02" width="0.1524" layer="91"/>
 <wire x1="76.2" y1="33.02" x2="76.2" y2="27.94" width="0.1524" layer="91"/>

Commit message: fixed lib
Connections:
- net DSG: now also M1.GATE; no longer M1.G
- net GND_OUT: now also M1.DRAIN_2; no longer M1.D
- net SRP: now also M1.SOURCE_2; no longer M1.S@2
Changed lines of the file:
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@@
 <part name="C14" library="pie" deviceset="CAP_POL" device="RADIAL" value="10uF"/>
 <part name="J3" library="SparkFun-Connectors" deviceset="USB_B" device="_PTH"/>
-<part name="M1" library="pie" deviceset="NMOS_CSD17579Q3A" device=""/>
 <part name="STANDOFF1" library="pie" deviceset="STAND-OFF" device="TIGHT"/>
 <part name="STANDOFF2" library="pie" deviceset="STAND-OFF" device="TIGHT"/>
@@
 <part name="STANDOFF7" library="pie" deviceset="STAND-OFF" device="TIGHT"/>
 <part name="C17" library="pie" deviceset="CAP" device="0603-CAP" value="2.2uF"/>
+<part name="M1" library="pie" deviceset="NMOS_CSD17579Q3A" device=""/>
 </parts>
 <sheets>
@@
 <attribute name="VALUE" x="-73.66" y="76.2" size="1.778" layer="96" rot="R270"/>
 </instance>
-<instance part="M1" gate="A" x="76.2" y="22.86" smashed="yes">
-<attribute name="NAME" x="81.28" y="22.86" size="1.778" layer="95"/>
-<attribute name="VALUE" x="81.28" y="20.32" size="1.778" layer="96"/>
-</instance>
 <instance part="STANDOFF1" gate="G$1" x="-109.22" y="86.36" smashed="yes"/>
 <instance part="STANDOFF2" gate="G$1" x="-99.06" y="86.36" smashed="yes"/>
@@
 <attribute name="NAME" x="-78.74" y="-21.59" size="1.778" layer="95" rot="R90"/>
 <attribute name="VALUE" x="-71.12" y="-21.59" size="1.778" layer="96" rot="R90"/>
+</instance>
+<instance part="M1" gate="A" x="71.12" y="25.4" smashed="yes">
+<attribute name="NAME" x="63.8556" y="31.9786" size="2.0828" layer="95" ratio="6" rot="SR0"/>
+<attribute name="VALUE" x="63.2206" y="29.4386" size="2.0828" layer="96" ratio="6" rot="SR0"/>
 </instance>
 </instances>
@@
 <label x="-20.32" y="15.24" size="1.778" layer="95"/>
 <wire x1="-20.32" y1="25.4" x2="66.04" y2="25.4" width="0.1524" layer="91"/>
-<wire x1="66.04" y1="25.4" x2="68.58" y2="25.4" width="0.1524" layer="91"/>
 <wire x1="66.04" y1="25.4" x2="66.04" y2="-10.16" width="0.1524" layer="91"/>
+<pinref part="R6" gate="G$1" pin="2"/>
+<pinref part="M1" gate="A" pin="GATE"/>
+<wire x1="66.04" y1="25.4" x2="67.31" y2="25.4" width="0.1524" layer="91"/>
 <junction x="66.04" y="25.4"/>
-<pinref part="R6" gate="G$1" pin="2"/>
-<pinref part="M1" gate="A" pin="G"/>
-<wire x1="68.58" y1="25.4" x2="68.58" y2="20.32" width="0.1524" layer="91"/>
 </segment>
 </net>
@@
 <pinref part="R7" gate="G$1" pin="2"/>
 <junction x="76.2" y="7.62"/>
-<pinref part="M1" gate="A" pin="S@2"/>
+<pinref part="M1" gate="A" pin="SOURCE_2"/>
+<wire x1="76.2" y1="17.78" x2="74.93" y2="17.78" width="0.1524" layer="91"/>
 </segment>
 </net>
@@
 <wire x1="73.66" y1="38.1" x2="76.2" y2="38.1" width="0.1524" layer="91"/>
 <label x="71.12" y="38.1" size="1.778" layer="95"/>
-<pinref part="M1" gate="A" pin="D"/>
-<wire x1="73.66" y1="33.02" x2="76.2" y2="33.02" width="0.1524" layer="91"/>
-<wire x1="76.2" y1="33.02" x2="76.2" y2="27.94" width="0.1524" layer="91"/>
-</segment>
-<segment>
+<pinref part="M1" gate="A" pin="DRAIN_2"/>
+<wire x1="73.66" y1="33.02" x2="74.93" y2="33.02" width="0.1524" layer="91"/>
+</segment>
+<segment>

Commit message: gerbs
Parts:
- M1: MANUFACTURER_PART_NUMBER (none) -> CSD16401Q5
- renumbered LS2 to BUZ1
Changed lines of the file:
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@@
 <grid distance="0.1" unitdist="inch" unit="inch" style="lines" multiple="1" display="no" altdistance="0.01" altunitdist="inch" altunit="inch"/>
 <layers>
-<layer number="1" name="Top" color="4" fill="1" visible="no" active="no"/>
-<layer number="2" name="Route2" color="16" fill="1" visible="no" active="no"/>
-<layer number="3" name="Route3" color="17" fill="1" visible="no" active="no"/>
-<layer number="4" name="Route4" color="18" fill="1" visible="no" active="no"/>
-<layer number="5" name="Route5" color="19" fill="1" visible="no" active="no"/>
-<layer number="6" name="Route6" color="25" fill="1" visible="no" active="no"/>
-<layer number="7" name="Route7" color="26" fill="1" visible="no" active="no"/>
-<layer number="8" name="Route8" color="27" fill="1" visible="no" active="no"/>
-<layer number="9" name="Route9" color="28" fill="1" visible="no" active="no"/>
-<layer number="10" name="Route10" color="29" fill="1" visible="no" active="no"/>
-<layer number="11" name="Route11" color="30" fill="1" visible="no" active="no"/>
-<layer number="12" name="Route12" color="20" fill="1" visible="no" active="no"/>
-<layer number="13" name="Route13" color="21" fill="1" visible="no" active="no"/>
-<layer number="14" name="Route14" color="22" fill="1" visible="no" active="no"/>
-<layer number="15" name="Route15" color="23" fill="1" visible="no" active="no"/>
-<layer number="16" name="Bottom" color="1" fill="1" visible="no" active="no"/>
-<layer number="17" name="Pads" color="2" fill="1" visible="no" active="no"/>
-<layer number="18" name="Vias" color="2" fill="1" visible="no" active="no"/>
-<layer number="19" name="Unrouted" color="6" fill="1" visible="no" active="no"/>
-<layer number="20" name="Dimension" color="24" fill="1" visible="no" active="no"/>
-<layer number="21" name="tPlace" color="7" fill="1" visible="no" active="no"/>
-<layer number="22" name="bPlace" color="7" fill="1" visible="no" active="no"/>
-<layer number="23" name="tOrigins" color="15" fill="1" visible="no" active="no"/>
-<layer number="24" name="bOrigins" color="15" fill="1" visible="no" active="no"/>
-<layer number="25" name="tNames" color="7" fill="1" visible="no" active="no"/>
-<layer number="26" name="bNames" color="7" fill="1" visible="no" active="no"/>
-<layer number="27" name="tValues" color="7" fill="1" visible="no" active="no"/>
-<layer number="28" name="bValues" color="7" fill="1" visible="no" active="no"/>
+<layer number="1" name="Top" color="4" fill="1" visible="yes" active="no"/>
+<layer number="2" name="Route2" color="16" fill="1" visible="yes" active="no"/>
+<layer number="3" name="Route3" color="17" fill="1" visible="yes" active="no"/>
+<layer number="4" name="Route4" color="18" fill="1" visible="yes" active="no"/>
+<layer number="5" name="Route5" color="19" fill="1" visible="yes" active="no"/>
+<layer number="6" name="Route6" color="25" fill="1" visible="yes" active="no"/>
+<layer number="7" name="Route7" color="26" fill="1" visible="yes" active="no"/>
+<layer number="8" name="Route8" color="27" fill="1" visible="yes" active="no"/>
+<layer number="9" name="Route9" color="28" fill="1" visible="yes" active="no"/>
+<layer number="10" name="Route10" color="29" fill="1" visible="yes" active="no"/>
+<layer number="11" name="Route11" color="30" fill="1" visible="yes" active="no"/>
+<layer number="12" name="Route12" color="20" fill="1" visible="yes" active="no"/>
+<layer number="13" name="Route13" color="21" fill="1" visible="yes" active="no"/>
+<layer number="14" name="Route14" color="22" fill="1" visible="yes" active="no"/>
+<layer number="15" name="Route15" color="23" fill="1" visible="yes" active="no"/>
+<layer number="16" name="Bottom" color="1" fill="1" visible="yes" active="no"/>
+<layer number="17" name="Pads" color="2" fill="1" visible="yes" active="no"/>
+<layer number="18" name="Vias" color="2" fill="1" visible="yes" active="no"/>
+<layer number="19" name="Unrouted" color="6" fill="1" visible="yes" active="no"/>
+<layer number="20" name="Dimension" color="24" fill="1" visible="yes" active="no"/>
+<layer number="21" name="tPlace" color="7" fill="1" visible="yes" active="no"/>
+<layer number="22" name="bPlace" color="7" fill="1" visible="yes" active="no"/>
+<layer number="23" name="tOrigins" color="15" fill="1" visible="yes" active="no"/>
+<layer number="24" name="bOrigins" color="15" fill="1" visible="yes" active="no"/>
+<layer number="25" name="tNames" color="7" fill="1" visible="yes" active="no"/>
+<layer number="26" name="bNames" color="7" fill="1" visible="yes" active="no"/>
+<layer number="27" name="tValues" color="7" fill="1" visible="yes" active="no"/>
+<layer number="28" name="bValues" color="7" fill="1" visible="yes" active="no"/>
 <layer number="29" name="tStop" color="7" fill="3" visible="no" active="no"/>
 <layer number="30" name="bStop" color="7" fill="6" visible="no" active="no"/>
@@
 <layer number="35" name="tGlue" color="7" fill="4" visible="no" active="no"/>
 <layer number="36" name="bGlue" color="7" fill="5" visible="no" active="no"/>
-<layer number="37" name="tTest" color="7" fill="1" visible="no" active="no"/>
-<layer number="38" name="bTest" color="7" fill="1" visible="no" active="no"/>
+<layer number="37" name="tTest" color="7" fill="1" visible="yes" active="no"/>
+<layer number="38" name="bTest" color="7" fill="1" visible="yes" active="no"/>
 <layer number="39" name="tKeepout" color="4" fill="11" visible="no" active="no"/>
 <layer number="40" name="bKeepout" color="1" fill="11" visible="no" active="no"/>
@@
 <layer number="44" name="Drills" color="7" fill="1" visible="no" active="no"/>
 <layer number="45" name="Holes" color="7" fill="1" visible="no" active="no"/>
-<layer number="46" name="Milling" color="3" fill="1" visible="no" active="no"/>
-<layer number="47" name="Measures" color="7" fill="1" visible="no" active="no"/>
-<layer number="48" name="Document" color="7" fill="1" visible="no" active="no"/>
-<layer number="49" name="Reference" color="7" fill="1" visible="no" active="no"/>
-<layer number="50" name="dxf" color="7" fill="1" visible="no" active="no"/>
-<layer number="51" name="tDocu" color="7" fill="1" visible="no" active="no"/>
-<layer number="52" name="bDocu" color="7" fill="1" visible="no" active="no"/>
-<layer number="53" name="tGND_GNDA" color="7" fill="9" visible="no" active="no"/>
-<layer number="54" name="bGND_GNDA" color="1" fill="9" visible="no" active="no"/>
-<layer number="56" name="wert" color="7" fill="1" visible="no" active="no"/>
-<layer number="57" name="tCAD" color="7" fill="1" visible="no" active="no"/>
-<layer number="59" name="tCarbon" color="7" fill="1" visible="no" active="no"/>
-<layer number="60" name="bCarbon" color="7" fill="1" visible="no" active="no"/>
+<layer number="46" name="Milling" color="3" fill="1" visible="yes" active="no"/>
+<layer number="47" name="Measures" color="7" fill="1" visible="yes" active="no"/>
+<layer number="48" name="Document" color="7" fill="1" visible="yes" active="no"/>
+<layer number="49" name="Reference" color="7" fill="1" visible="yes" active="no"/>
+<layer number="50" name="dxf" color="7" fill="1" visible="yes" active="no"/>
+<layer number="51" name="tDocu" color="7" fill="1" visible="yes" active="no"/>
+<layer number="52" name="bDocu" color="7" fill="1" visible="yes" active="no"/>
+<layer number="53" name="tGND_GNDA" color="7" fill="9" visible="yes" active="no"/>
+<layer number="54" name="bGND_GNDA" color="1" fill="9" visible="yes" active="no"/>
+<layer number="56" name="wert" color="7" fill="1" visible="yes" active="no"/>
+<layer number="57" name="tCAD" color="7" fill="1" visible="yes" active="no"/>
+<layer number="59" name="tCarbon" color="7" fill="1" visible="yes" active="no"/>
+<layer number="60" name="bCarbon" color="7" fill="1" visible="yes" active="no"/>
 <layer number="88" name="SimResults" color="9" fill="1" visible="yes" active="yes"/>
 <layer number="89" name="SimProbes" color="9" fill="1" visible="yes" active="yes"/>
@@
 <part name="R28" library="pie" deviceset="R-US_" device="R0603" value="22R"/>
 <part name="R29" library="pie" deviceset="R-US_" device="R0603" value="22R"/>
-<part name="LS2" library="pie" deviceset="BUZZER" device="3.3VBUZZER"/>
+<part name="BUZ1" library="pie" deviceset="BUZZER" device="3.3VBUZZER"/>
 <part name="J2" library="pie" deviceset="AVR_SPI_PRG_6" device="MA03-2"/>
 <part name="SUPPLY18" library="pie" deviceset="GND" device=""/>
@@
 <part name="STANDOFF7" library="pie" deviceset="STAND-OFF" device="TIGHT"/>
 <part name="C17" library="pie" deviceset="CAP" device="0603-CAP" value="2.2uF"/>
-<part name="M1" library="pie" deviceset="NMOS_CSD17579Q3A" device=""/>
+<part name="M1" library="pie" deviceset="NMOS_CSD17579Q3A" device="" value="">
+<attribute name="MANUFACTURER_PART_NUMBER" value="CSD16401Q5"/>
+</part>
 </parts>
 <sheets>
@@
 <attribute name="VALUE" x="-43.18" y="-29.21" size="1.778" layer="96"/>
 </instance>
-<instance part="LS2" gate="G$1" x="71.12" y="10.16" smashed="yes">
+<instance part="BUZ1" gate="G$1" x="71.12" y="10.16" smashed="yes">
 <attribute name="NAME" x="66.04" y="15.24" size="1.778" layer="95"/>
 <attribute name="VALUE" x="66.04" y="2.54" size="1.778" layer="96"/>
@@
 <segment>
 <pinref part="SUPPLY13" gate="GND" pin="GND"/>
-<pinref part="LS2" gate="G$1" pin="C"/>
+<pinref part="BUZ1" gate="G$1" pin="C"/>
 </segment>
 <segment>
@@
 <label x="43.18" y="12.7" size="1.778" layer="95"/>
 <wire x1="40.64" y1="12.7" x2="66.04" y2="12.7" width="0.1524" layer="91"/>
-<pinref part="LS2" gate="G$1" pin="A"/>
-</segment>
-</net>
+<pinref part="BUZ1" gate="G$1" pin="A"/>
+</segment>
+</net>
