File: Boards/PDB2/PDB/PDB2_1.sch (EAGLE design)
At the start: 78 parts, among them J1 XT60CONNECTOR, J2 AVR_SPI_PRG_6MA03-2, J3 USB_B_PTH, M1 NMOS_CSD17579Q3A, SW1 PUSH_BUTTON, U1 BQ7692006PWRPW20-M, U2 Value, U3 ATMEGA32U4-AU

Commit message: fixed pdb drc
Changed lines of the file:
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@@
 <grid distance="0.1" unitdist="inch" unit="inch" style="lines" multiple="1" display="no" altdistance="0.01" altunitdist="inch" altunit="inch"/>
 <layers>
-<layer number="1" name="Top" color="4" fill="1" visible="yes" active="no"/>
-<layer number="2" name="Route2" color="16" fill="1" visible="yes" active="no"/>
-<layer number="3" name="Route3" color="17" fill="1" visible="yes" active="no"/>
-<layer number="4" name="Route4" color="18" fill="1" visible="yes" active="no"/>
-<layer number="5" name="Route5" color="19" fill="1" visible="yes" active="no"/>
-<layer number="6" name="Route6" color="25" fill="1" visible="yes" active="no"/>
-<layer number="7" name="Route7" color="26" fill="1" visible="yes" active="no"/>
-<layer number="8" name="Route8" color="27" fill="1" visible="yes" active="no"/>
-<layer number="9" name="Route9" color="28" fill="1" visible="yes" active="no"/>
-<layer number="10" name="Route10" color="29" fill="1" visible="yes" active="no"/>
-<layer number="11" name="Route11" color="30" fill="1" visible="yes" active="no"/>
-<layer number="12" name="Route12" color="20" fill="1" visible="yes" active="no"/>
-<layer number="13" name="Route13" color="21" fill="1" visible="yes" active="no"/>
-<layer number="14" name="Route14" color="22" fill="1" visible="yes" active="no"/>
-<layer number="15" name="Route15" color="23" fill="1" visible="yes" active="no"/>
-<layer number="16" name="Bottom" color="1" fill="1" visible="yes" active="no"/>
-<layer number="17" name="Pads" color="2" fill="1" visible="yes" active="no"/>
-<layer number="18" name="Vias" color="2" fill="1" visible="yes" active="no"/>
-<layer number="19" name="Unrouted" color="6" fill="1" visible="yes" active="no"/>
-<layer number="20" name="Dimension" color="24" fill="1" visible="yes" active="no"/>
-<layer number="21" name="tPlace" color="7" fill="1" visible="yes" active="no"/>
-<layer number="22" name="bPlace" color="7" fill="1" visible="yes" active="no"/>
-<layer number="23" name="tOrigins" color="15" fill="1" visible="yes" active="no"/>
-<layer number="24" name="bOrigins" color="15" fill="1" visible="yes" active="no"/>
-<layer number="25" name="tNames" color="7" fill="1" visible="yes" active="no"/>
-<layer number="26" name="bNames" color="7" fill="1" visible="yes" active="no"/>
-<layer number="27" name="tValues" color="7" fill="1" visible="yes" active="no"/>
-<layer number="28" name="bValues" color="7" fill="1" visible="yes" active="no"/>
+<layer number="1" name="Top" color="4" fill="1" visible="no" active="no"/>
+<layer number="2" name="Route2" color="16" fill="1" visible="no" active="no"/>
+<layer number="3" name="Route3" color="17" fill="1" visible="no" active="no"/>
+<layer number="4" name="Route4" color="18" fill="1" visible="no" active="no"/>
+<layer number="5" name="Route5" color="19" fill="1" visible="no" active="no"/>
+<layer number="6" name="Route6" color="25" fill="1" visible="no" active="no"/>
+<layer number="7" name="Route7" color="26" fill="1" visible="no" active="no"/>
+<layer number="8" name="Route8" color="27" fill="1" visible="no" active="no"/>
+<layer number="9" name="Route9" color="28" fill="1" visible="no" active="no"/>
+<layer number="10" name="Route10" color="29" fill="1" visible="no" active="no"/>
+<layer number="11" name="Route11" color="30" fill="1" visible="no" active="no"/>
+<layer number="12" name="Route12" color="20" fill="1" visible="no" active="no"/>
+<layer number="13" name="Route13" color="21" fill="1" visible="no" active="no"/>
+<layer number="14" name="Route14" color="22" fill="1" visible="no" active="no"/>
+<layer number="15" name="Route15" color="23" fill="1" visible="no" active="no"/>
+<layer number="16" name="Bottom" color="1" fill="1" visible="no" active="no"/>
+<layer number="17" name="Pads" color="2" fill="1" visible="no" active="no"/>
+<layer number="18" name="Vias" color="2" fill="1" visible="no" active="no"/>
+<layer number="19" name="Unrouted" color="6" fill="1" visible="no" active="no"/>
+<layer number="20" name="Dimension" color="24" fill="1" visible="no" active="no"/>
+<layer number="21" name="tPlace" color="7" fill="1" visible="no" active="no"/>
+<layer number="22" name="bPlace" color="7" fill="1" visible="no" active="no"/>
+<layer number="23" name="tOrigins" color="15" fill="1" visible="no" active="no"/>
+<layer number="24" name="bOrigins" color="15" fill="1" visible="no" active="no"/>
+<layer number="25" name="tNames" color="7" fill="1" visible="no" active="no"/>
+<layer number="26" name="bNames" color="7" fill="1" visible="no" active="no"/>
+<layer number="27" name="tValues" color="7" fill="1" visible="no" active="no"/>
+<layer number="28" name="bValues" color="7" fill="1" visible="no" active="no"/>
 <layer number="29" name="tStop" color="7" fill="3" visible="no" active="no"/>
 <layer number="30" name="bStop" color="7" fill="6" visible="no" active="no"/>
@@
 <layer number="35" name="tGlue" color="7" fill="4" visible="no" active="no"/>
 <layer number="36" name="bGlue" color="7" fill="5" visible="no" active="no"/>
-<layer number="37" name="tTest" color="7" fill="1" visible="yes" active="no"/>
-<layer number="38" name="bTest" color="7" fill="1" visible="yes" active="no"/>
+<layer number="37" name="tTest" color="7" fill="1" visible="no" active="no"/>
+<layer number="38" name="bTest" color="7" fill="1" visible="no" active="no"/>
 <layer number="39" name="tKeepout" color="4" fill="11" visible="no" active="no"/>
 <layer number="40" name="bKeepout" color="1" fill="11" visible="no" active="no"/>
@@
 <layer number="44" name="Drills" color="7" fill="1" visible="no" active="no"/>
 <layer number="45" name="Holes" color="7" fill="1" visible="no" active="no"/>
-<layer number="46" name="Milling" color="3" fill="1" visible="yes" active="no"/>
-<layer number="47" name="Measures" color="7" fill="1" visible="yes" active="no"/>
-<layer number="48" name="Document" color="7" fill="1" visible="yes" active="no"/>
-<layer number="49" name="Reference" color="7" fill="1" visible="yes" active="no"/>
-<layer number="50" name="dxf" color="7" fill="1" visible="yes" active="no"/>
-<layer number="51" name="tDocu" color="7" fill="1" visible="yes" active="no"/>
-<layer number="52" name="bDocu" color="7" fill="1" visible="yes" active="no"/>
-<layer number="53" name="tGND_GNDA" color="7" fill="9" visible="yes" active="no"/>
-<layer number="54" name="bGND_GNDA" color="1" fill="9" visible="yes" active="no"/>
-<layer number="56" name="wert" color="7" fill="1" visible="yes" active="no"/>
-<layer number="57" name="tCAD" color="7" fill="1" visible="yes" active="no"/>
-<layer number="59" name="tCarbon" color="7" fill="1" visible="yes" active="no"/>
-<layer number="60" name="bCarbon" color="7" fill="1" visible="yes" active="no"/>
+<layer number="46" name="Milling" color="3" fill="1" visible="no" active="no"/>
+<layer number="47" name="Measures" color="7" fill="1" visible="no" active="no"/>
+<layer number="48" name="Document" color="7" fill="1" visible="no" active="no"/>
+<layer number="49" name="Reference" color="7" fill="1" visible="no" active="no"/>
+<layer number="50" name="dxf" color="7" fill="1" visible="no" active="no"/>
+<layer number="51" name="tDocu" color="7" fill="1" visible="no" active="no"/>
+<layer number="52" name="bDocu" color="7" fill="1" visible="no" active="no"/>
+<layer number="53" name="tGND_GNDA" color="7" fill="9" visible="no" active="no"/>
+<layer number="54" name="bGND_GNDA" color="1" fill="9" visible="no" active="no"/>
+<layer number="56" name="wert" color="7" fill="1" visible="no" active="no"/>
+<layer number="57" name="tCAD" color="7" fill="1" visible="no" active="no"/>
+<layer number="59" name="tCarbon" color="7" fill="1" visible="no" active="no"/>
+<layer number="60" name="bCarbon" color="7" fill="1" visible="no" active="no"/>
 <layer number="88" name="SimResults" color="9" fill="1" visible="yes" active="yes"/>
 <layer number="89" name="SimProbes" color="9" fill="1" visible="yes" active="yes"/>
@@
 <part name="STANDOFF7" library="pie" deviceset="STAND-OFF" device="TIGHT"/>
 <part name="C17" library="pie" deviceset="CAP" device="0603-CAP" value="2.2uF"/>
-<part name="M1" library="pie" deviceset="NMOS_CSD17579Q3A" device="" value="">
+<part name="M1" library="pie" deviceset="NMOS_CSD17579Q3A" device="" value="NMOS_CSD17579Q3A">
 <attribute name="MANUFACTURER_PART_NUMBER" value="CSD16401Q5"/>
 </part>

Commit message: please no mere conflict
Parts:
- removed C17: 2.2uF, pie:CAP0603-CAP
- removed R29: 22R, pie:R-US_R0603
- added D1: D_NRVB120VLSFT1G, pie:D_NRVB120VLSFT1G
- added D3: BZT52C2VXX_ZENER, pie:BZT52C2VXX_ZENER
- added R9: 56.2k, pie:R-US_R0603
- C10: value 1uF -> 22uF; device pie:CAP0603-CAP -> resistor:C-USC0805
- C11: value 10uF -> 22uF; device pie:CAP_POLRADIAL -> resistor:C-USC0805
- C12: value 18pF -> 2.2uF
- C14: value 10uF -> 18pF; device pie:CAP_POLRADIAL -> pie:CAP0603-CAP
- C15, C16, C2: value 1uF -> 2.2uF
- C4: value .1uF -> 2.2uF
- C5: value 10uF -> .1uF; device pie:CAP0805 -> pie:CAP0603-CAP
- C6: value 10uF -> 22uF
- C7: value 8.2nF -> 22uF; device pie:CAP0603-CAP -> pie:CAP0805
- C9: value 47uF -> 22uF; device pie:CAP0805 -> resistor:C-USC0805
- D2: value D_MBR1020VL -> BZT52C2VXX_ZENER; device pie:D_MBR1020VL -> pie:BZT52C2VXX_ZENER
- J2: value AVR_SPI_PRG_6MA03-2 -> USB_B_PTH; device pie:AVR_SPI_PRG_6MA03-2 -> SparkFun-Connectors:USB_B_PTH
- J3: value USB_B_PTH -> AVR_SPI_PRG_6MA03-2; device SparkFun-Connectors:USB_B_PTH -> pie:AVR_SPI_PRG_6MA03-2
- L1: device pie:L_VLP8040T-3R3N -> pie:MWSA0420S_INDUCTORMW
- M1: value NMOS_CSD17579Q3A -> CSD17577Q3A; MANUFACTURER_PART_NUMBER CSD16401Q5 -> CSD17577Q3A
- R10: value 56.2k -> 10k
- R11, R12: value 10k -> 22R
- R13: value 220R -> 10k
- R14, R15, R16, R17: value 220R -> 330R
- R18: value 150R -> 330R
- R19, R20, R21, R22, R23, R24, R25, R26, R27: value 150R -> 220R
- R28: value 22R -> 220R
- R5: value 499k -> 100k
- R7: device pie:SHUNT_SMD -> pie:R-US_R2512; MANUFACTURER_PART_NO WSHM28185L000FEA -> (none)
- U2: value Value -> (none); device pie:TPS563210ADDFR -> pie:TPS563200
- Y1: value (none) -> 8MHZ_X50328MSB2GI; device pie:CRYSTAL10.5X4.8 -> pie:8MHZ_X50328MSB2GI; PART_NO ECS-160-20-3X-EN-TR -> (none)
- renumbered JP7 to JP6, STANDOFF7 to STANDOFF6
Connections:
- removed net N$9: C7.2, U2.SS
- net 12V: now also C7.2, D1.A, D2.N; no longer C5.2, D2.A
- net 3.3V: now also C4.2; no longer C3.2
- net 5V: now also C10.1, C11.1, C9.1, D3.N, L1.1, R9.2; no longer C11.+, C14.+, C9.2, L1.2, R10.2
- net CAP1: now also C3.2; no longer C2.2
- net D+: now also J2.D+, R11.1; no longer J3.D+, R29.1
- net D-: now also J2.D-, R12.1; no longer J3.D-, R28.1
- net EN/MISO: now also J3.1; no longer J2.1
- net FB: now also R10.2, R9.1; no longer R10.1, R11.2
- net GND: now also C14.1, C4.1, C5.2, J2.GND, J2.SHIELD, J3.6, R7.2; no longer C10.1, C17.1, C4.2, J2.6, J3.GND, J3.SHIELD, R7.1
- net GND_OUT: now also C10.2, C11.2, C9.2, D2.P, D3.P, R10.1; no longer C11.-, C14.-, C5.1, C9.1, R11.1
- net LED1: now also R28.1; no longer R27.1
- net LED10: now also R19.1; no longer R18.1
- net LED2: now also R27.1; no longer R26.1
- net LED3: now also R26.1; no longer R25.1
- net LED4: now also R25.1; no longer R24.1
- net LED5: now also R24.1; no longer R23.1
- net LED6: now also R23.1; no longer R22.1
- net LED7: now also R22.1; no longer R21.1
- net LED8: now also R21.1; no longer R20.1
- net LED9: now also R20.1; no longer R19.1
- net MOSI: now also J3.4; no longer J2.4
- net N$12: now also R19.2; no longer R18.2
- net N$13: now also R20.2; no longer R19.2
- net N$14: now also R21.2; no longer R20.2
- net N$15: now also R22.2; no longer R21.2
- net N$16: now also R23.2; no longer R22.2
- net N$17: now also R24.2; no longer R23.2
- net N$18: now also R25.2; no longer R24.2
- net N$19: now also R26.2; no longer R25.2
- net N$2: now also C13.2; no longer C12.2
- net N$20: now also R27.2; no longer R26.2
- net N$21: now also R28.2; no longer R27.2
- net N$22: now also R18.1; no longer R17.1
- net N$23: now also R18.2; no longer R17.2
- net N$24: now also R14.2; no longer R13.2
- net N$25: now also R14.1; no longer R13.1
- net N$28: now also R17.1; no longer R16.1
- net N$29: now also R16.1; no longer R15.1
- net N$3: now also R12.2; no longer R28.2
- net N$30: now also R15.1; no longer R14.1
- net N$31: now also R17.2; no longer R16.2
- net N$32: now also R16.2; no longer R15.2
- net N$33: now also R15.2; no longer R14.2
- net N$4: now also R11.2; no longer R29.2
- net N$5: now also C14.2; no longer C13.2
- net RST: now also J3.5, R13.1; no longer J2.5, R12.1
- net SCLK: now also J3.3; no longer J2.3
- net SRP: now also C5.1, R7.1; no longer C4.1, R7.2
- net SW: now also L1.2; no longer L1.1
- net UVCC: now also C12.2, J2.VBUS, J3.2; no longer C10.2, J2.2, J3.VBUS
- net VCC: now also R13.2; no longer R12.2
- net VIN: now also C2.2, D1.C; no longer C17.2, D2.C
Other:
- moved on the sheet: C1, C12, C13, C2, C3, C4, C6, C7, C9, R10, R12, R13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
