File: Boards/TI_MotorController/TI_MotorController/TI_MotorController.sch (EAGLE design)
At the start: 37 parts, among them J1 CONN_12X2, M1 NMOS_CSD17579Q3A, M2 NMOS_CSD17579Q3A, M3 NMOS_CSD17579Q3A, M4 NMOS_CSD17579Q3A, M5 NMOS_CSD17579Q3A, M6 NMOS_CSD17579Q3A, M7 NMOS_CSD17579Q3A, M8 NMOS_CSD17579Q3A, U1 DRV8704, U2 ATMEGA32U4-AU

Commit message: Slight modification
Connections:
- net N$13 renamed AISENP
Changed lines of the file:
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@@
 <?xml version="1.0" encoding="utf-8"?>
 <!DOCTYPE eagle SYSTEM "eagle.dtd">
-<eagle version="9.3.0">
+<eagle version="9.4.2">
 <drawing>
 <settings>
@@
 </segment>
 </net>
-<net name="N$13" class="0">
+<net name="AISENP" class="0">
 <segment>
 <pinref part="U1" gate="G$1" pin="AISENP"/>
@@
 <pinref part="M4" gate="A" pin="S@2"/>
 <pinref part="M2" gate="A" pin="S@2"/>
-</segment>
-</net>
+<label x="127" y="17.78" size="1.778" layer="95"/>
+</segment>
+</net>

Commit message: thweou th
Connections:
- new net N$9: C6.1, C7.1, C8.1, C9.1, U2.(HWB)PE2, U2.GND, U2.GND2, U2.GND3, U2.GND4, U2.UGND
- net GND: no longer C6.1, C7.1, C8.1, C9.1, U2.(HWB)PE2, U2.GND, U2.GND2, U2.GND3, U2.GND4, U2.UGND
Other:
- moved on the sheet: J1
