File: Boards/MotorControllerV2/MotorControllerV2.sch (EAGLE design)
At the start: 45 parts, among them J1 CONN_12X2, M10 NMOS_CSD17579Q3A, M11 NMOS_CSD17579Q3A, M12 NMOS_CSD17579Q3A, M13 NMOS_CSD17579Q3A, M14 NMOS_CSD17579Q3A, M15 NMOS_CSD17579Q3A, M16 NMOS_CSD17579Q3A, M9 NMOS_CSD17579Q3A, U2 ATMEGA32U4-AU, U3 DRV8704

Commit message: Continued working on new motor controller
Parts:
- removed C7: 18pF, pie:CAP0603-CAP
- removed C8: 1uF, pie:CAP0603-CAP
- added C4: 1uF, pie:CAP0603-CAP
- added C5: 18pF, pie:CAP0603-CAP
- added J2: USB_B_PTH, SparkFun-Connectors:USB_B_PTH
- renumbered C16 to C2, C17 to C3, C9 to C1
Connections:
- net D+: now also C2.2, J2.D+; no longer C3.2
- net D-: now also C3.2, J2.D-; no longer C2.2
- net GND: now also C4.1, C5.1, J2.GND, J2.SHIELD; no longer C7.1, C8.1
- net N$3: now also R1.1; no longer R1.2
- net N$7: now also C6.2; no longer C7.2
- net N$8: now also C5.2; no longer C6.2
- net VCC: now also C4.2, J2.VBUS, R1.2; no longer C8.2, R1.1
Other:
- moved on the sheet: C6, R1

Commit message: Continuing work
Parts:
- removed J1: CONN_12X2, SparkFun-Connectors:CONN_12X2
- added U$2: 12PIN, pie:12PIN
- renumbered M10 to M2, M11 to M3, M12 to M4, M13 to M5, M14 to M6, M15 to M7, M16 to M8, M9 to M1
Connections:
- net N$10 renamed VINT
- net N$12 renamed V5
- net N$13 renamed VCP
- net N$14 renamed CP2
- net N$15 renamed CP1
- removed net AIN1M: J1.6, U3.AIN1
- removed net AIN2M: J1.8, U3.AIN2
- removed net BIN1M: J1.10, U3.BIN1
- removed net BIN2M: J1.12, U3.BIN2
- removed net FAULTNM: J1.22, R5.2, U3.FAULTN
- removed net RESETM: J1.4, U3.RESET
- removed net SCLKM: J1.14, U3.SCLK
- removed net SCSM: J1.18, U3.SCS
- removed net SDATIM: J1.16, U3.SDATI
- removed net SDATOM: J1.20, U3.SDATO
- removed net SLEEPM: J1.2, U3.SLEEPN
- net A1: now also U2.(TXD1/INT3)PD3; no longer U2.(PCINT6/OC1B/OC4B/ADC13)PB6
- net AIN1: now also U3.AIN1; no longer J1.5
- net AIN2: now also U3.AIN2; no longer J1.7
- net B1: now also U2.(ADC7/TDI)PF7; no longer U2.(TXD1/INT3)PD3
- net BIN1: now also U3.BIN1; no longer J1.9
- net BIN2: now also U3.BIN2; no longer J1.11
- net BISENN: no longer C18.1, C19.1, C20.1, C21.1, U3.GND, U3.GND2, U3.GND3, U3.GND4, U3.GND_PAD
- net FAULTN: now also R5.2, U3.FAULTN; no longer J1.21
- net GND: now also C18.1, C19.1, C20.1, C21.1, U3.GND, U3.GND2, U3.GND3, U3.GND4, U3.GND_PAD; no longer J1.23, J1.24
- net LED1: now also U2.(ADC4/TCK)PF4; no longer U2.(ADC5/TMS)PF5
- net LED2: now also U2.(ADC1)PF1; no longer U2.(ADC6/TDO)PF6
- net LED3: now also U2.(ADC0)PF0; no longer U2.(ADC7/TDI)PF7
- net RESET: now also U2.(PCINT6/OC1B/OC4B/ADC13)PB6, U3.RESET; no longer J1.3, U2.(PCINT4/ADC11)PB4
- net SCLK: now also U3.SCLK; no longer J1.13
- net SCS: now also U3.SCS; no longer J1.17
- net SDATI: now also U3.SDATI; no longer J1.15
- net SDATO: now also U3.SDATO; no longer J1.19
- net SLEEP: now also U3.SLEEPN; no longer J1.1

Commit message: fixerd
Connections:
- removed net AISENN: R6.1, U3.AISENN
- removed net BISENN: R7.1, U3.BISENN
- net GND: now also R6.1, R7.1, U3.AISENN, U3.BISENN
Changed lines of the file:
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@@
 <?xml version="1.0" encoding="utf-8"?>
 <!DOCTYPE eagle SYSTEM "eagle.dtd">
-<eagle version="9.4.2">
+<eagle version="9.3.0">
 <drawing>
 <settings>
@@
 <part name="SUPPLY9" library="pie" deviceset="GND" device=""/>
 <part name="SUPPLY10" library="pie" deviceset="GND" device=""/>
-<part name="SUPPLY11" library="pie" deviceset="GND" device=""/>
 <part name="SUPPLY12" library="pie" deviceset="GND" device=""/>
 <part name="SUPPLY13" library="pie" deviceset="GND" device=""/>
@@
 <part name="C6" library="pie" deviceset="CAP" device="0603-CAP" value="18pF"/>
 <part name="U$2" library="pie" deviceset="12PIN" device=""/>
+<part name="SUPPLY3" library="pie" deviceset="GND" device=""/>
+<part name="SUPPLY4" library="pie" deviceset="GND" device=""/>
+<part name="SUPPLY7" library="pie" deviceset="GND" device=""/>
 </parts>
 <sheets>
@@
 <attribute name="VALUE" x="158.75" y="74.93" size="1.778" layer="96"/>
 </instance>
-<instance part="SUPPLY11" gate="GND" x="116.84" y="-10.16" smashed="yes">
-<attribute name="VALUE" x="115.57" y="-13.97" size="1.778" layer="96"/>
-</instance>
 <instance part="SUPPLY12" gate="GND" x="142.24" y="10.16" smashed="yes">
 <attribute name="VALUE" x="140.97" y="6.35" size="1.778" layer="96"/>
@@
 <instance part="CONN3" gate="G$1" x="25.4" y="106.68" smashed="yes" rot="MR180">
 <attribute name="NAME" x="17.78" y="100.584" size="1.778" layer="95" rot="MR180"/>
+</instance>
+<instance part="SUPPLY3" gate="GND" x="142.24" y="10.16" smashed="yes">
+<attribute name="VALUE" x="140.97" y="6.35" size="1.778" layer="96"/>
+</instance>
+<instance part="SUPPLY4" gate="GND" x="116.84" y="-10.16" smashed="yes">
+<attribute name="VALUE" x="115.57" y="-13.97" size="1.778" layer="96"/>
+</instance>
+<instance part="SUPPLY7" gate="GND" x="119.38" y="58.42" smashed="yes">
+<attribute name="VALUE" x="118.11" y="54.61" size="1.778" layer="96"/>
 </instance>
 </instances>
@@
 </segment>
 </net>
-<net name="BISENN" class="0">
-<segment>
-<pinref part="U3" gate="G$1" pin="BISENN"/>
-<wire x1="60.96" y1="7.62" x2="55.88" y2="7.62" width="0.1524" layer="91"/>
-<label x="58.42" y="7.62" size="1.778" layer="95"/>
-</segment>
-<segment>
-<pinref part="R7" gate="G$1" pin="1"/>
-<wire x1="116.84" y1="-7.62" x2="106.68" y2="-7.62" width="0.1524" layer="91"/>
-<label x="106.68" y="-7.62" size="1.778" layer="95"/>
-<pinref part="SUPPLY11" gate="GND" pin="GND"/>
-<junction x="116.84" y="-7.62"/>
-</segment>
-</net>
-<net name="AISENN" class="0">
-<segment>
-<pinref part="R6" gate="G$1" pin="1"/>
-<wire x1="109.22" y1="60.96" x2="119.38" y2="60.96" width="0.1524" layer="91"/>
-<label x="109.22" y="60.96" size="1.778" layer="95"/>
-</segment>
-<segment>
-<pinref part="U3" gate="G$1" pin="AISENN"/>
-<wire x1="55.88" y1="30.48" x2="60.96" y2="30.48" width="0.1524" layer="91"/>
-<label x="58.42" y="30.48" size="1.778" layer="95"/>
-</segment>
-</net>
 <net name="GND" class="0">
 <segment>
@@
 <pinref part="C26" gate="G$1" pin="-"/>
 <wire x1="142.24" y1="12.7" x2="142.24" y2="17.78" width="0.1524" layer="91"/>
+<pinref part="SUPPLY3" gate="GND" pin="GND"/>
+<junction x="142.24" y="12.7"/>
 </segment>
 <segment>
@@
 <label x="12.7" y="-25.4" size="1.778" layer="95"/>
 </segment>
-</net>
+<segment>
+<pinref part="R7" gate="G$1" pin="1"/>
+<pinref part="SUPPLY4" gate="GND" pin="GND"/>
+</segment>
+<segment>
+<pinref part="R6" gate="G$1" pin="1"/>
+<pinref part="SUPPLY7" gate="GND" pin="GND"/>
+</segment>
+<segment>
+<pinref part="U3" gate="G$1" pin="AISENN"/>
+<wire x1="55.88" y1="30.48" x2="60.96" y2="30.48" width="0.1524" layer="91"/>
+<label x="58.42" y="30.48" size="1.778" layer="95"/>
+</segment>
+<segment>
+<pinref part="U3" gate="G$1" pin="BISENN"/>
+<wire x1="60.96" y1="7.62" x2="55.88" y2="7.62" width="0.1524" layer="91"/>
+<label x="58.42" y="7.62" size="1.778" layer="95"/>
+</segment>
+</net>

Commit message: Rev A
Connections:
- net A1: now also R8.8; no longer R8.6
- net A2: now also R8.6; no longer R8.8
- net B1: now also R8.7; no longer R8.5
- net B2: now also R8.5; no longer R8.7
Other:
- moved on the sheet: ENC1, ENC2
Changed lines of the file:
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@@
 <?xml version="1.0" encoding="utf-8"?>
 <!DOCTYPE eagle SYSTEM "eagle.dtd">
-<eagle version="9.3.0">
+<eagle version="9.4.2">
 <drawing>
 <settings>
@@
 <attribute name="VALUE" x="69.85" y="72.39" size="1.778" layer="96"/>
 </instance>
-<instance part="ENC1" gate="G$1" x="5.08" y="35.56" smashed="yes">
-<attribute name="VALUE" x="2.54" y="25.4" size="1.778" layer="96"/>
-<attribute name="NAME" x="2.54" y="41.91" size="1.778" layer="95"/>
+<instance part="ENC1" gate="G$1" x="7.62" y="22.86" smashed="yes">
+<attribute name="VALUE" x="5.08" y="12.7" size="1.778" layer="96"/>
+<attribute name="NAME" x="5.08" y="29.21" size="1.778" layer="95"/>
 </instance>
 <instance part="R8" gate="G$1" x="43.18" y="17.78" smashed="yes">
@@
 <attribute name="VALUE" x="33.02" y="12.7" size="3.81" layer="94" font="vector"/>
 </instance>
-<instance part="ENC2" gate="G$1" x="5.08" y="17.78" smashed="yes">
-<attribute name="VALUE" x="2.54" y="7.62" size="1.778" layer="96"/>
-<attribute name="NAME" x="2.54" y="24.13" size="1.778" layer="95"/>
+<instance part="ENC2" gate="G$1" x="7.62" y="40.64" smashed="yes">
+<attribute name="VALUE" x="5.08" y="30.48" size="1.778" layer="96"/>
+<attribute name="NAME" x="5.08" y="46.99" size="1.778" layer="95"/>
 </instance>
 <instance part="FRAME1" gate="G$1" x="-157.48" y="-66.04" smashed="yes"/>
@@
 <segment>
 <pinref part="ENC1" gate="G$1" pin="2"/>
-<wire x1="12.7" y1="33.02" x2="17.78" y2="33.02" width="0.1524" layer="91"/>
-<label x="12.7" y="33.02" size="1.778" layer="95"/>
+<wire x1="15.24" y1="20.32" x2="20.32" y2="20.32" width="0.1524" layer="91"/>
+<label x="15.24" y="20.32" size="1.778" layer="95"/>
 </segment>
 <segment>
 <pinref part="ENC2" gate="G$1" pin="2"/>
-<wire x1="12.7" y1="15.24" x2="17.78" y2="15.24" width="0.1524" layer="91"/>
-<label x="12.7" y="15.24" size="1.778" layer="95"/>
+<wire x1="15.24" y1="38.1" x2="20.32" y2="38.1" width="0.1524" layer="91"/>
+<label x="15.24" y="38.1" size="1.778" layer="95"/>
 </segment>
 <segment>
@@
 <segment>
 <pinref part="ENC1" gate="G$1" pin="1"/>
-<wire x1="12.7" y1="30.48" x2="17.78" y2="30.48" width="0.1524" layer="91"/>
-<label x="12.7" y="30.48" size="1.778" layer="95"/>
+<wire x1="15.24" y1="17.78" x2="20.32" y2="17.78" width="0.1524" layer="91"/>
+<label x="15.24" y="17.78" size="1.778" layer="95"/>
 </segment>
 <segment>
@@
 <segment>
 <pinref part="ENC2" gate="G$1" pin="1"/>
-<wire x1="12.7" y1="12.7" x2="17.78" y2="12.7" width="0.1524" layer="91"/>
-<label x="12.7" y="12.7" size="1.778" layer="95"/>
+<wire x1="15.24" y1="35.56" x2="20.32" y2="35.56" width="0.1524" layer="91"/>
+<label x="15.24" y="35.56" size="1.778" layer="95"/>
 </segment>
 <segment>
@@
 <net name="A1" class="0">
 <segment>
-<pinref part="ENC1" gate="G$1" pin="3"/>
-<pinref part="R8" gate="G$1" pin="6"/>
-<wire x1="30.48" y1="35.56" x2="12.7" y2="35.56" width="0.1524" layer="91"/>
-<label x="12.7" y="35.56" size="1.778" layer="95"/>
-</segment>
-<segment>
 <pinref part="U2" gate="G$1" pin="(TXD1/INT3)PD3"/>
 <wire x1="-25.4" y1="2.54" x2="-20.32" y2="2.54" width="0.1524" layer="91"/>
 <label x="-22.86" y="2.54" size="1.778" layer="95"/>
 </segment>
+<segment>
+<pinref part="ENC1" gate="G$1" pin="3"/>
+<wire x1="15.24" y1="22.86" x2="30.48" y2="22.86" width="0.1524" layer="91"/>
+<pinref part="R8" gate="G$1" pin="8"/>
+<wire x1="30.48" y1="22.86" x2="30.48" y2="20.32" width="0.1524" layer="91"/>
+<label x="15.24" y="22.86" size="1.778" layer="95"/>
+</segment>
 </net>
 <net name="B1" class="0">
 <segment>
 <pinref part="ENC1" gate="G$1" pin="4"/>
-<wire x1="12.7" y1="38.1" x2="17.78" y2="38.1" width="0.1524" layer="91"/>
-<pinref part="R8" gate="G$1" pin="5"/>
-<wire x1="30.48" y1="43.18" x2="17.78" y2="43.18" width="0.1524" layer="91"/>
-<wire x1="17.78" y1="43.18" x2="17.78" y2="38.1" width="0.1524" layer="91"/>
-<label x="12.7" y="38.1" size="1.778" layer="95"/>
+<label x="15.24" y="25.4" size="1.778" layer="95"/>
+<pinref part="R8" gate="G$1" pin="7"/>
+<wire x1="15.24" y1="25.4" x2="30.48" y2="25.4" width="0.1524" layer="91"/>
+<wire x1="30.48" y1="25.4" x2="30.48" y2="27.94" width="0.1524" layer="91"/>
 </segment>
 <segment>
@@
 <segment>
 <pinref part="ENC2" gate="G$1" pin="3"/>
-<wire x1="12.7" y1="17.78" x2="27.94" y2="17.78" width="0.1524" layer="91"/>
-<wire x1="27.94" y1="17.78" x2="27.94" y2="20.32" width="0.1524" layer="91"/>
-<pinref part="R8" gate="G$1" pin="8"/>
-<wire x1="27.94" y1="20.32" x2="30.48" y2="20.32" width="0.1524" layer="91"/>
-<label x="12.7" y="17.78" size="1.778" layer="95"/>
+<wire x1="15.24" y1="40.64" x2="30.48" y2="40.64" width="0.1524" layer="91"/>
+<label x="15.24" y="40.64" size="1.778" layer="95"/>
+<pinref part="R8" gate="G$1" pin="6"/>
+<wire x1="30.48" y1="40.64" x2="30.48" y2="35.56" width="0.1524" layer="91"/>
 </segment>
 <segment>
@@
 <segment>
 <pinref part="ENC2" gate="G$1" pin="4"/>
-<wire x1="12.7" y1="20.32" x2="20.32" y2="20.32" width="0.1524" layer="91"/>
-<wire x1="20.32" y1="20.32" x2="20.32" y2="27.94" width="0.1524" layer="91"/>
-<pinref part="R8" gate="G$1" pin="7"/>
-<wire x1="20.32" y1="27.94" x2="30.48" y2="27.94" width="0.1524" layer="91"/>
-<label x="12.7" y="20.32" size="1.778" layer="95"/>
-</segment>
-<segment>
+<label x="15.24" y="43.18" size="1.778" layer="95"/>
+<pinref part="R8" gate="G$1" pin="5"/>
+<wire x1="15.24" y1="43.18" x2="30.48" y2="43.18" width="0.1524" layer="91"/>
+</segment>
+<segment>

Commit message: isp pls
Parts:
- removed U$2: 12PIN, pie:12PIN
Changed lines of the file:
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@@
 <part name="C5" library="pie" deviceset="CAP" device="0603-CAP" value="18pF"/>
 <part name="C6" library="pie" deviceset="CAP" device="0603-CAP" value="18pF"/>
-<part name="U$2" library="pie" deviceset="12PIN" device=""/>
 <part name="SUPPLY3" library="pie" deviceset="GND" device=""/>
 <part name="SUPPLY4" library="pie" deviceset="GND" device=""/>
@@
 <attribute name="NAME" x="-115.57" y="17.78" size="1.778" layer="95"/>
 <attribute name="VALUE" x="-115.57" y="10.16" size="1.778" layer="96"/>
-</instance>
-<instance part="U$2" gate="G$1" x="-144.78" y="93.98" smashed="yes">
-<attribute name="NAME" x="-142.24" y="104.14" size="1.27" layer="94" font="vector"/>
 </instance>
 </instances>
@@
 <segment>
 <pinref part="U3" gate="G$1" pin="A1HS"/>
-<wire x1="55.88" y1="38.1" x2="60.96" y2="38.1" width="0.1524" layer="91"/>
 <label x="58.42" y="38.1" size="1.778" layer="95"/>
+<wire x1="55.88" y1="38.1" x2="76.2" y2="38.1" width="0.1524" layer="91"/>
 </segment>
 <segment>
@@
 <segment>
 <pinref part="U3" gate="G$1" pin="AILS"/>
-<wire x1="55.88" y1="35.56" x2="60.96" y2="35.56" width="0.1524" layer="91"/>
 <label x="58.42" y="35.56" size="1.778" layer="95"/>
+<wire x1="55.88" y1="35.56" x2="76.2" y2="35.56" width="0.1524" layer="91"/>
 </segment>
 <segment>
@@
 <segment>
 <pinref part="U3" gate="G$1" pin="A2LS"/>
-<wire x1="55.88" y1="27.94" x2="60.96" y2="27.94" width="0.1524" layer="91"/>
 <label x="58.42" y="27.94" size="1.778" layer="95"/>
+<wire x1="55.88" y1="27.94" x2="76.2" y2="27.94" width="0.1524" layer="91"/>
 </segment>
 <segment>
@@
 <segment>
 <pinref part="U3" gate="G$1" pin="AOUT2"/>
-<wire x1="55.88" y1="22.86" x2="60.96" y2="22.86" width="0.1524" layer="91"/>
 <label x="58.42" y="22.86" size="1.778" layer="95"/>
+<wire x1="55.88" y1="22.86" x2="76.2" y2="22.86" width="0.1524" layer="91"/>
 </segment>
 <segment>
@@
 <segment>
 <pinref part="U3" gate="G$1" pin="AOUT1"/>
-<wire x1="55.88" y1="40.64" x2="60.96" y2="40.64" width="0.1524" layer="91"/>
 <label x="58.42" y="40.64" size="1.778" layer="95"/>
+<wire x1="55.88" y1="40.64" x2="76.2" y2="40.64" width="0.1524" layer="91"/>
 </segment>
 <segment>
@@
 <segment>
 <pinref part="U3" gate="G$1" pin="A2HS"/>
-<wire x1="55.88" y1="25.4" x2="60.96" y2="25.4" width="0.1524" layer="91"/>
 <label x="58.42" y="25.4" size="1.778" layer="95"/>
+<wire x1="55.88" y1="25.4" x2="76.2" y2="25.4" width="0.1524" layer="91"/>
 </segment>
 <segment>
@@
 <segment>
 <pinref part="U3" gate="G$1" pin="BOUT1"/>
-<wire x1="55.88" y1="17.78" x2="60.96" y2="17.78" width="0.1524" layer="91"/>
 <label x="58.42" y="17.78" size="1.778" layer="95"/>
+<wire x1="55.88" y1="17.78" x2="76.2" y2="17.78" width="0.1524" layer="91"/>
 </segment>
 <segment>
@@
 <segment>
 <pinref part="U3" gate="G$1" pin="BOUT2"/>
-<wire x1="55.88" y1="0" x2="60.96" y2="0" width="0.1524" layer="91"/>
 <label x="58.42" y="0" size="1.778" layer="95"/>
+<wire x1="55.88" y1="0" x2="76.2" y2="0" width="0.1524" layer="91"/>
 </segment>
 <segment>
@@
 <segment>
 <pinref part="U3" gate="G$1" pin="B1HS"/>
-<wire x1="55.88" y1="15.24" x2="60.96" y2="15.24" width="0.1524" layer="91"/>
 <label x="58.42" y="15.24" size="1.778" layer="95"/>
+<wire x1="55.88" y1="15.24" x2="76.2" y2="15.24" width="0.1524" layer="91"/>
 </segment>
 </net>
@@
 <segment>
 <pinref part="U3" gate="G$1" pin="B1LS"/>
-<wire x1="55.88" y1="12.7" x2="60.96" y2="12.7" width="0.1524" layer="91"/>
 <label x="58.42" y="12.7" size="1.778" layer="95"/>
+<wire x1="55.88" y1="12.7" x2="76.2" y2="12.7" width="0.1524" layer="91"/>
 </segment>
 </net>
@@
 <segment>
 <pinref part="U3" gate="G$1" pin="B2HS"/>
-<wire x1="55.88" y1="2.54" x2="60.96" y2="2.54" width="0.1524" layer="91"/>
 <label x="58.42" y="2.54" size="1.778" layer="95"/>
+<wire x1="55.88" y1="2.54" x2="76.2" y2="2.54" width="0.1524" layer="91"/>
 </segment>
 </net>
@@
 <segment>
 <pinref part="U3" gate="G$1" pin="B2LS"/>
-<wire x1="55.88" y1="5.08" x2="60.96" y2="5.08" width="0.1524" layer="91"/>
 <label x="58.42" y="5.08" size="1.778" layer="95"/>
+<wire x1="55.88" y1="5.08" x2="76.2" y2="5.08" width="0.1524" layer="91"/>
 </segment>
 </net>
@@
 <segment>
 <pinref part="U3" gate="G$1" pin="BISENP"/>
-<wire x1="55.88" y1="10.16" x2="60.96" y2="10.16" width="0.1524" layer="91"/>
 <label x="58.42" y="10.16" size="1.778" layer="95"/>
-</segment>
-<segment>
+<wire x1="55.88" y1="10.16" x2="66.04" y2="10.16" width="0.1524" layer="91"/>
+</segment>
+<segment>

Commit message: isp pls
Parts:
- added J1: AVR_SPI_PRG_6MA03-2, pie:AVR_SPI_PRG_6MA03-2
Connections:
- net GND: now also J1.6
- net RESET: now also J1.5
- net SCLK: now also J1.3
- net SDATI: now also J1.4
- net SDATO: now also J1.1
- net VCC: now also J1.2
Changed lines of the file:
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@@
 <part name="SUPPLY4" library="pie" deviceset="GND" device=""/>
 <part name="SUPPLY7" library="pie" deviceset="GND" device=""/>
+<part name="J1" library="pie" deviceset="AVR_SPI_PRG_6" device="MA03-2"/>
 </parts>
 <sheets>
@@
 <attribute name="NAME" x="-115.57" y="17.78" size="1.778" layer="95"/>
 <attribute name="VALUE" x="-115.57" y="10.16" size="1.778" layer="96"/>
+</instance>
+<instance part="J1" gate="G$1" x="-43.18" y="81.28" smashed="yes">
+<attribute name="NAME" x="-48.26" y="87.63" size="1.778" layer="95"/>
+<attribute name="VALUE" x="-48.26" y="73.66" size="1.778" layer="96"/>
 </instance>
 </instances>
@@
 <label x="-119.38" y="40.64" size="1.778" layer="95"/>
 </segment>
+<segment>
+<pinref part="J1" gate="G$1" pin="6"/>
+<wire x1="-33.02" y1="78.74" x2="-22.86" y2="78.74" width="0.1524" layer="91"/>
+<label x="-27.94" y="78.74" size="1.778" layer="95"/>
+</segment>
 </net>
 <net name="SLEEP" class="0">
@@
 <label x="-22.86" y="25.4" size="1.778" layer="95"/>
 </segment>
+<segment>
+<pinref part="J1" gate="G$1" pin="5"/>
+<wire x1="-50.8" y1="78.74" x2="-58.42" y2="78.74" width="0.1524" layer="91"/>
+<label x="-60.96" y="78.74" size="1.778" layer="95"/>
+</segment>
 </net>
 <net name="AIN1" class="0">
@@
 <label x="-22.86" y="38.1" size="1.778" layer="95"/>
 </segment>
+<segment>
+<pinref part="J1" gate="G$1" pin="3"/>
+<wire x1="-50.8" y1="81.28" x2="-58.42" y2="81.28" width="0.1524" layer="91"/>
+<label x="-60.96" y="81.28" size="1.778" layer="95"/>
+</segment>
 </net>
 <net name="SDATI" class="0">
@@
 <label x="-22.86" y="35.56" size="1.778" layer="95"/>
 </segment>
+<segment>
+<pinref part="J1" gate="G$1" pin="4"/>
+<wire x1="-33.02" y1="81.28" x2="-22.86" y2="81.28" width="0.1524" layer="91"/>
+<label x="-27.94" y="81.28" size="1.778" layer="95"/>
+</segment>
 </net>
 <net name="SCS" class="0">
@@
 <wire x1="-25.4" y1="33.02" x2="-17.78" y2="33.02" width="0.1524" layer="91"/>
 <label x="-22.86" y="33.02" size="1.778" layer="95"/>
+</segment>
+<segment>
+<pinref part="J1" gate="G$1" pin="1"/>
+<wire x1="-50.8" y1="83.82" x2="-58.42" y2="83.82" width="0.1524" layer="91"/>
+<label x="-60.96" y="83.82" size="1.778" layer="95"/>
 </segment>
 </net>
@@
 <label x="58.42" y="20.32" size="1.778" layer="95"/>
 </segment>
-</net>
+<segment>
+<pinref part="J1" gate="G$1" pin="2"/>
+<wire x1="-33.02" y1="83.82" x2="-22.86" y2="83.82" width="0.1524" layer="91"/>
+<label x="-27.94" y="83.82" size="1.778" layer="95"/>
+</segment>
+</net>

Commit message: fixed
Connections:
- removed net N$3: R1.1, U2.RESET
- new net RST: J1.5, R1.1, U2.RESET
- net RESET: no longer J1.5
Changed lines of the file:
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@@
 <label x="-22.86" y="25.4" size="1.778" layer="95"/>
-</segment>
-<segment>
-<pinref part="J1" gate="G$1" pin="5"/>
-<wire x1="-50.8" y1="78.74" x2="-58.42" y2="78.74" width="0.1524" layer="91"/>
-<label x="-60.96" y="78.74" size="1.778" layer="95"/>
 </segment>
 </net>
@@
 </segment>
 </net>
-<net name="N$3" class="0">
+<net name="RST" class="0">
 <segment>
 <pinref part="U2" gate="G$1" pin="RESET"/>
 <wire x1="-83.82" y1="45.72" x2="-88.9" y2="45.72" width="0.1524" layer="91"/>
 <pinref part="R1" gate="G$1" pin="1"/>
-</segment>
-</net>
+<label x="-88.9" y="43.18" size="1.778" layer="95"/>
+</segment>
+<segment>
+<pinref part="J1" gate="G$1" pin="5"/>
+<wire x1="-50.8" y1="78.74" x2="-58.42" y2="78.74" width="0.1524" layer="91"/>
+<label x="-60.96" y="78.74" size="1.778" layer="95"/>
+</segment>
+</net>
