File: Boards/Ultrasonic_IR/Breakout/breakout.brd (EAGLE design)
At the start: 78 x 50.5 mm, 3 parts, among them IC1 ARDUINO_PRO_MICRO

Commit message: usir files
Parts:
- added U$2: (no value), pie:OSHW-LOGO-S
- added U$3: (no value), pie:PIE-LOGO-SMALL
Routing:
- net GND: track 5.85 -> 0.00 mm, vias 3 -> 1
- net OUT: track 29.1 -> 28.2 mm
Other:
- board text added: "(c) Pioneers In Engineering Design by: Kaitlyn, Erica, Aryaman This design is open source hardware. For more information, visit pioneers.berkeley.edu/opensource"
- board text added: "ULTRASONIC + IR BREAKOUT"
Changed lines of the file:
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@@
 <setting verticaltext="up"/>
 </settings>
-<grid distance="19.6850394" unitdist="mil" unit="mil" style="lines" multiple="1" display="yes" altdistance="5" altunitdist="mil" altunit="mil"/>
+<grid distance="1" unitdist="mm" unit="mm" style="lines" multiple="1" display="yes" altdistance="5" altunitdist="mil" altunit="mil"/>
 <layers>
 <layer number="1" name="Top" color="4" fill="1" visible="yes" active="yes"/>
@@
 <text x="24.5" y="42.5" size="1.778" layer="25" font="vector" rot="R180">VCC</text>
 <text x="16.5" y="34.5" size="1.778" layer="25" font="vector" rot="R90">GND</text>
+<text x="38.585" y="1.142" size="1.27" layer="22" font="vector" rot="MR0">(c) Pioneers In Engineering
+Design by: Kaitlyn, Erica, Aryaman
+This design is open source hardware.
+For more information, visit
+pioneers.berkeley.edu/opensource</text>
+<text x="73" y="48" size="1.778" layer="21" font="vector" rot="R270">ULTRASONIC + IR BREAKOUT</text>
 </plain>
 <attributes>
@@
 <attribute name="REFERENCE_DEST" value="ARDUINO_PRO_MICRO" x="29.5" y="45.5" size="1.778" layer="27" rot="R270" display="off"/>
 </element>
+<element name="U$2" library="pie" package="OSHW-LOGO-S" value="" x="3.5" y="3" smashed="yes"/>
+<element name="U$3" library="pie" package="PIE-LOGO-SMALL" value="" x="7.5" y="14.5" smashed="yes"/>
 </elements>
 <signals>
 <signal name="OUT">
 <contactref element="U$1" pad="3"/>
-<wire x1="13.12" y1="42" x2="12.5" y2="42.62" width="0.1524" layer="1"/>
 <contactref element="IC1" pad="10"/>
 <wire x1="13.12" y1="42" x2="13.12" y2="34.38" width="0.3048" layer="1"/>
@@
 <contactref element="IC1" pad="GND@2"/>
 <contactref element="IC1" pad="GND@1"/>
-<wire x1="55.81" y1="15" x2="55.81" y2="16.81" width="0.3048" layer="1"/>
-<wire x1="55.81" y1="16.81" x2="56.5" y2="17.5" width="0.3048" layer="1"/>
-<via x="56.5" y="17.5" extent="1-16" drill="0.381"/>
-<wire x1="15.66" y1="42" x2="15.66" y2="44.84" width="0.3048" layer="1"/>
-<wire x1="15.66" y1="44.84" x2="15.5" y2="45" width="0.3048" layer="1"/>
-<via x="15.5" y="45" extent="1-16" drill="0.381"/>
 </signal>
 <signal name="VCC">
@@
 </board>
 </drawing>
+<compatibility>
+<note version="6.3" minversion="6.2.2" severity="warning">
+Since Version 6.2.2 text objects can contain more than one line,
+which will not be processed correctly with this version.
+</note>
+</compatibility>
 </eagle>

Commit message: ultrasonic
Parts:
- removed U$2: (no value), pie:OSHW-LOGO-S
- added LED1: RED, pie:LED-1206
- added LED2: YELLOW, pie:LED-1206
- added LED3: GREEN, pie:LED-1206
- added R2: 330, pie:4X-0603
- moved U$3 62.8 mm to (69.5, 4.50)
- moved IC1 11.4 mm to (36.5, 36.5)
Connections:
- new net LED1: IC1.A1, LED1.A
- new net LED2: IC1.A0, LED2.A
- new net LED3: IC1.15, LED3.A
- new net N$1: LED2.C, R2.6
- new net N$2: LED1.C, R2.5
- new net N$6: LED3.C, R2.7
- net GND: now also R2.2, R2.3, R2.4
Routing:
- net VCC: track 94.5 -> 0.00 mm, vias 2 -> 0
- net OUT: track 28.2 -> 0.00 mm
- net ECHO: track 24.9 -> 0.00 mm
- net TRIG: track 24.4 -> 0.00 mm
Other:
- board size 78 x 50.5 mm -> 78 x 45.5 mm
