File: Boards/Ultrasonic_IR/Breakout/breakout.sch (EAGLE design)
At the start: 3 parts, among them IC1 ARDUINO_PRO_MICRO

Commit message: usir files
Other:
- note added: "11/25/19"
- note added: "Ultrasonic/IR Breakout"
- moved on the sheet: IC1

Commit message: ultrasonic
Parts:
- added LED1: RED, pie:LED1206
- added LED2: YELLOW, pie:LED1206
- added LED3: GREEN, pie:LED1206
- added R2: 330, pie:4X-0603
Connections:
- new net LED1: IC1.A1, LED1.A
- new net LED2: IC1.A0, LED2.A
- new net LED3: IC1.15, LED3.A
- new net N$1: LED2.C, R2.6
- new net N$2: LED1.C, R2.5
- new net N$6: LED3.C, R2.7
- net GND: now also R2.2, R2.3, R2.4
Changed lines of the file:
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@@
 <part name="IC1" library="pie" deviceset="ARDUINO_PRO_MICRO" device=""/>
 <part name="FRAME1" library="pie" deviceset="FRAME_SCHEMATIC" device=""/>
+<part name="LED1" library="pie" deviceset="LED" device="1206" value="RED"/>
+<part name="SUPPLY6" library="pie" deviceset="GND" device=""/>
+<part name="LED2" library="pie" deviceset="LED" device="1206" value="YELLOW"/>
+<part name="SUPPLY7" library="pie" deviceset="GND" device=""/>
+<part name="LED3" library="pie" deviceset="LED" device="1206" value="GREEN"/>
+<part name="SUPPLY8" library="pie" deviceset="GND" device=""/>
+<part name="R2" library="pie" deviceset="4X-0603" device="" value="330"/>
 </parts>
 <sheets>
@@
 <attribute name="SHEET" x="124.46" y="-59.69" size="2.54" layer="94" font="vector"/>
 </instance>
+<instance part="LED1" gate="G$1" x="-38.1" y="96.52" smashed="yes">
+<attribute name="NAME" x="-41.91" y="99.06" size="1.778" layer="95"/>
+<attribute name="VALUE" x="-41.91" y="90.17" size="1.778" layer="96"/>
+</instance>
+<instance part="SUPPLY6" gate="GND" x="15.24" y="86.36" smashed="yes">
+<attribute name="VALUE" x="13.97" y="82.55" size="1.778" layer="96"/>
+</instance>
+<instance part="LED2" gate="G$1" x="-38.1" y="81.28" smashed="yes">
+<attribute name="NAME" x="-41.91" y="83.82" size="1.778" layer="95"/>
+<attribute name="VALUE" x="-41.91" y="74.93" size="1.778" layer="96"/>
+</instance>
+<instance part="SUPPLY7" gate="GND" x="15.24" y="78.74" smashed="yes">
+<attribute name="VALUE" x="13.97" y="74.93" size="1.778" layer="96"/>
+</instance>
+<instance part="LED3" gate="G$1" x="-38.1" y="66.04" smashed="yes">
+<attribute name="NAME" x="-41.91" y="68.58" size="1.778" layer="95"/>
+<attribute name="VALUE" x="-41.91" y="59.69" size="1.778" layer="96"/>
+</instance>
+<instance part="SUPPLY8" gate="GND" x="15.24" y="93.98" smashed="yes">
+<attribute name="VALUE" x="13.97" y="90.17" size="1.778" layer="96"/>
+</instance>
+<instance part="R2" gate="G$1" x="-5.08" y="71.12" smashed="yes">
+<attribute name="NAME" x="-12.7" y="101.6" size="3.81" layer="94" font="vector"/>
+<attribute name="VALUE" x="-15.24" y="66.04" size="3.81" layer="94" font="vector"/>
+</instance>
 </instances>
 <busses>
@@
 <pinref part="IC1" gate="APM" pin="GND@1"/>
 </segment>
+<segment>
+<pinref part="SUPPLY6" gate="GND" pin="GND"/>
+<wire x1="7.62" y1="88.9" x2="15.24" y2="88.9" width="0.1524" layer="91"/>
+<pinref part="R2" gate="G$1" pin="3"/>
+</segment>
+<segment>
+<pinref part="SUPPLY7" gate="GND" pin="GND"/>
+<wire x1="7.62" y1="81.28" x2="15.24" y2="81.28" width="0.1524" layer="91"/>
+<pinref part="R2" gate="G$1" pin="2"/>
+</segment>
+<segment>
+<pinref part="R2" gate="G$1" pin="4"/>
+<pinref part="SUPPLY8" gate="GND" pin="GND"/>
+<wire x1="7.62" y1="96.52" x2="15.24" y2="96.52" width="0.1524" layer="91"/>
+</segment>
 </net>
 <net name="VCC" class="0">
@@
 </segment>
 </net>
+<net name="LED1" class="0">
+<segment>
+<pinref part="LED1" gate="G$1" pin="A"/>
+<wire x1="-40.64" y1="96.52" x2="-47.244" y2="96.52" width="0.1524" layer="91"/>
+<label x="-50.8" y="96.52" size="1.778" layer="95"/>
+</segment>
+<segment>
+<pinref part="IC1" gate="APM" pin="A1"/>
+<wire x1="-12.7" y1="22.86" x2="-10.16" y2="22.86" width="0.1524" layer="91"/>
+<label x="-7.62" y="22.86" size="1.778" layer="95"/>
+</segment>
+</net>
+<net name="LED2" class="0">
+<segment>
+<pinref part="LED2" gate="G$1" pin="A"/>
+<wire x1="-40.64" y1="81.28" x2="-47.244" y2="81.28" width="0.1524" layer="91"/>
+<label x="-50.8" y="81.28" size="1.778" layer="95"/>
+</segment>
+<segment>
+<pinref part="IC1" gate="APM" pin="A0"/>
+<wire x1="-12.7" y1="20.32" x2="-10.16" y2="20.32" width="0.1524" layer="91"/>
+<label x="-7.62" y="20.32" size="1.778" layer="95"/>
+</segment>
+</net>
+<net name="LED3" class="0">
+<segment>
+<pinref part="LED3" gate="G$1" pin="A"/>
+<wire x1="-40.64" y1="66.04" x2="-47.244" y2="66.04" width="0.1524" layer="91"/>
+<label x="-50.8" y="66.04" size="1.778" layer="95"/>
+</segment>
+<segment>
+<pinref part="IC1" gate="APM" pin="15"/>
+<wire x1="-12.7" y1="17.78" x2="-10.16" y2="17.78" width="0.1524" layer="91"/>
+<label x="-7.62" y="17.78" size="1.778" layer="95"/>
+</segment>
+</net>
+<net name="N$2" class="0">
+<segment>
+<pinref part="LED1" gate="G$1" pin="C"/>
+<wire x1="-35.56" y1="96.52" x2="-17.78" y2="96.52" width="0.1524" layer="91"/>
+<pinref part="R2" gate="G$1" pin="5"/>
+</segment>
+</net>
+<net name="N$6" class="0">
+<segment>
+<pinref part="LED3" gate="G$1" pin="C"/>
+<wire x1="-35.56" y1="66.04" x2="-22.86" y2="66.04" width="0.1524" layer="91"/>
+<pinref part="R2" gate="G$1" pin="7"/>
+<wire x1="-22.86" y1="66.04" x2="-22.86" y2="81.28" width="0.1524" layer="91"/>
+<wire x1="-22.86" y1="81.28" x2="-17.78" y2="81.28" width="0.1524" layer="91"/>
+</segment>
+</net>
+<net name="N$1" class="0">
+<segment>
+<pinref part="LED2" gate="G$1" pin="C"/>
+<wire x1="-35.56" y1="81.28" x2="-27.94" y2="81.28" width="0.1524" layer="91"/>
+<wire x1="-27.94" y1="81.28" x2="-27.94" y2="88.9" width="0.1524" layer="91"/>
+<pinref part="R2" gate="G$1" pin="6"/>
+<wire x1="-27.94" y1="88.9" x2="-17.78" y2="88.9" width="0.1524" layer="91"/>
+</segment>
+</net>
