File: Boards/LineFollower/LineFollowe/linefollower.sch (EAGLE design)
At the start: 9 parts, among them Q1 QRE1113, Q2 QRE1113, U1 LM358LVIDR

Commit message: line follower schematic
Parts:
- removed U$3: 5PIN, pie:5PIN
- added C2: 1mF, pie:CAP0402-CAP
- added C3: 10nF, pie:CAP0402-CAP
- added C4: 100nF, pie:CAP0402-CAP
- added C5: 0.1uF, pie:CAP0402-CAP
- added D1, D2, D3: (no value), pie:DIODESMA-ALT
- added IC1: ARDUINO_PRO_MICRO, pie:ARDUINO_PRO_MICRO
- added Q3, Q4, Q5, Q6: QRE1113, pie:QRE1113
- added R10, R11, R14, R15: 10k, pie:R-US_R0603
- added R12, R13, R8, R9: 1k, pie:R-US_R0603
- added R5, R6, R7: 330, pie:R-US_R0603
- added RF1, RF2, RF3, RF4, RF5, RF6: 1K, pie:R-US_R0603
- added R_GND, R_VCC: 100K, pie:R-US_R0603
- added R_LED1, R_LED2, R_LED3, R_LED4, R_LED5, R_LED6: 100, pie:R-US_R0603
- added U2, U3: AD8630ARUZ-REEL, pie:AD8630ARUZ-REEL
- C1: value (none) -> 10mF; device pie:CAP0603-CAP -> pie:CAP0402-CAP
- R1: value 100 -> 1k
- R2: value 100 -> 10k
- R3: value 5000 -> 1k
- R4: value 1000 -> 10k
- U1: value LM358LVIDR -> AD8630ARUZ-REEL; device pie:LM358LVIDR -> pie:AD8630ARUZ-REEL
Connections:
- removed net INV: C1.1, Q1.4, R3.2, U1.IN1-
- removed net VOUT: C1.2, R3.1, R4.1, U1.OUT1
- new net DIFF_1+: R3.2, R4.2, U1.+INC
- new net DIFF_1-: R1.2, R2.2, U1.-INC
- new net DIFF_2+: R10.2, R9.2, U2.+INC
- new net DIFF_2-: R11.2, R8.2, U2.-INC
- new net DIFF_3+: R13.2, R14.2, U3.+INC
- new net DIFF_3-: R12.2, R15.2, U3.-INC
- new net IRLED_EN: IC1.3
- new net IR_LED_1: IC1.A3, R_LED1.2, R_LED2.2
- new net IR_LED_2: IC1.A2, R_LED3.2, R_LED4.2
- new net IR_LED_3: IC1.15, R_LED5.2, R_LED6.2
- new net N$4: D2.A, R6.1
- new net N$7: Q4.1, R_LED4.1
- new net N$8: Q5.1, R_LED5.1
- new net N$9: Q6.1, R_LED6.1
- new net SENS_1: IC1.A1, R2.1, R5.2, U1.OUTC
- new net SENS_2: IC1.A0, R11.1, R6.2, U2.OUTC
- new net SENS_3: IC1.10, R15.1, R7.2, U3.OUTC
- new net TIA_1: Q1.3, RF1.1, U1.-INA
- new net TIA_2: Q2.3, RF2.2, U1.-INB
- new net TIA_3: Q3.3, RF3.1, U2.-INA
- new net TIA_4: Q4.3, RF4.2, U2.-INB
- new net TIA_5: Q5.3, RF5.1, U3.-INA
- new net TIA_6: Q6.3, RF6.2, U3.-INB
- new net VIR_GND: C5.2, R10.1, R14.1, R4.1, R_GND.2, R_VCC.1
- new net VO1_1: R1.1, RF1.2, U1.OUTA
- new net VO1_2: R8.1, RF3.2, U2.OUTA
- new net VO1_3: R12.1, RF5.2, U3.OUTA
- new net VO2_1: R3.1, RF2.1, U1.OUTB
- new net VO2_2: R9.1, RF4.1, U2.OUTB
- new net VO2_3: R13.1, RF6.1, U3.OUTB
- net GND: now also C1.2, C2.2, C3.2, C4.2, C5.1, D1.C, D2.C, D3.C, IC1.GND@0, IC1.GND@1, IC1.GND@2, Q1.4, Q2.4, Q3.2, Q3.4, Q4.2, Q4.4, Q5.2, Q5.4, Q6.2, Q6.4, R_GND.1, U1.+INA, U1.+INB, U2.+INA, U2.+INB, U2.V-, U3.+INA, U3.+INB, U3.V-; no longer Q1.3, Q2.3, U$3.GND, U1.IN1+
- net N$1: now also Q2.1, R_LED2.1; no longer R4.2, U$3.P1
- net N$2: now also D1.A, R5.1; no longer R1.2, U$3.P3
- net N$3: now also R_LED1.1; no longer R1.1
- net N$5: now also D3.A, R7.1; no longer Q2.1, R2.1
- net N$6: now also Q3.1, R_LED3.1; no longer R2.2, U$3.P2
- net VCC: now also C1.1, C2.1, C3.1, C4.1, IC1.VCC, R_VCC.2, U2.V+, U3.V+; no longer U$3.VCC
Other:
- note added: "TIAs (gain = RF = 1000)"
- note added: "decoupling caps"
- note added: "diff amp (gain = R2/R1 = 10)"
- note added: "photosensor output feedback"
- note added: "trigger IR LED"
- note added: "virtual ground to center diff amp around 2.5"
- moved on the sheet: C1, R1, R2, R3, R4

Commit message: added mux to line follower
Parts:
- removed D2, D3: (no value), pie:DIODESMA-ALT
- removed R10, R11, R14, R15: 10k, pie:R-US_R0603
- removed R12, R13, R8, R9: 1k, pie:R-US_R0603
- removed R6, R7: 330, pie:R-US_R0603
- removed RF3, RF4, RF5, RF6: 1K, pie:R-US_R0603
- removed U2, U3: AD8630ARUZ-REEL, pie:AD8630ARUZ-REEL
- added U4: 74VHC153FT(BJ), pie:74VHC153FT(BJ)
Connections:
- removed net DIFF_2+: R10.2, R9.2, U2.+INC
- removed net DIFF_2-: R11.2, R8.2, U2.-INC
- removed net DIFF_3+: R13.2, R14.2, U3.+INC
- removed net DIFF_3-: R12.2, R15.2, U3.-INC
- removed net IRLED_EN: IC1.3
- removed net N$4: D2.A, R6.1
- removed net N$5: D3.A, R7.1
- removed net SENS_2: IC1.A0, R11.1, R6.2, U2.OUTC
- removed net SENS_3: IC1.10, R15.1, R7.2, U3.OUTC
- removed net VO1_2: R8.1, RF3.2, U2.OUTA
- removed net VO1_3: R12.1, RF5.2, U3.OUTA
- removed net VO2_2: R9.1, RF4.1, U2.OUTB
- removed net VO2_3: R13.1, RF6.1, U3.OUTB
- new net CTRL_A: IC1.14, U4.14
- new net CTRL_B: IC1.16, U4.2
- new net N$18: U4.3
- new net N$23: U4.13
- new net STROBE_1: IC1.2, U4.1
- new net STROBE_2: IC1.3, U4.15
- new net TIA_A: RF1.1, U1.-INA, U4.7
- new net TIA_B: RF2.2, U1.-INB, U4.9
- net GND: now also U4.8; no longer D2.C, D3.C, U2.+INA, U2.+INB, U2.V-, U3.+INA, U3.+INB, U3.V-
- net TIA_1: now also U4.6; no longer RF1.1, U1.-INA
- net TIA_2: now also U4.10; no longer RF2.2, U1.-INB
- net TIA_3: now also U4.5; no longer RF3.1, U2.-INA
- net TIA_4: now also U4.11; no longer RF4.2, U2.-INB
- net TIA_5: now also U4.4; no longer RF5.1, U3.-INA
- net TIA_6: now also U4.12; no longer RF6.2, U3.-INB
- net VCC: now also U4.16; no longer U2.V+, U3.V+
- net VIR_GND: no longer R10.1, R14.1
Other:
- moved on the sheet: D1, R5

Commit message: lf updates
Parts:
- removed D1: (no value), pie:DIODESMA-ALT
- added LED1: RED, pie:LED0603
Connections:
- removed net N$18: U4.3
- removed net N$23: U4.13
- net GND: now also LED1.C, U4.13, U4.3; no longer D1.C
- net N$2: now also LED1.A; no longer D1.A
- net STROBE_1: now also IC1.A0; no longer IC1.2
- net STROBE_2: now also IC1.10; no longer IC1.3
Other:
- moved on the sheet: R5, R_LED3, R_LED4, R_LED5, R_LED6
