File: Boards/2020_MC_copy/mc.sch (EAGLE design)
At the start: 32 parts, among them J1 USB_B_PTH, J2 AVR_SPI_PRG_6MA03-2

Commit message: 2/17 mc2020 update
Parts:
- removed U$1: 32U4, pie:ATMEGA32U4QFN
- added C10, C11, C12, C9: 0.1 uF, pie:CAP0402-CAP
- added C13, C14: LELON_ELECTROLYTIC_CAP, pie:LELON_ELECTROLYTIC_CAP
- added U1: 32U4, pie:ATMEGA32U4QFN
- C7: value (none) -> 1 uF
- LED1, LED2, LED3, LED4, LED5: device pie:LED1206 -> pie:LED0805
- R4: value (none) -> 330
- R5: value (none) -> 10k
- Y1: device pie:CRYSTAL10.5X4.8 -> pie:CRYSTAL
- renumbered MC_A to MC1, MC_B to MC2
Connections:
- net A1: now also U1.PD3(TX); no longer U$1.PD3(TX)
- net A2: now also U1.PF7(ADC7); no longer U$1.PF7(ADC7)
- net AIN1: now also U1.PC6; no longer U$1.PC6
- net AIN2: now also U1.PB5(ADC12); no longer U$1.PB5(ADC12)
- net B1: now also U1.PD1(SDA); no longer U$1.PD1(SDA)
- net B2: now also U1.PD2(RX); no longer U$1.PD2(RX)
- net BIN1: now also U1.PD7(ADC10); no longer U$1.PD7(ADC10)
- net BIN2: now also U1.PD0(SCL); no longer U$1.PD0(SCL)
- net FAULT_N: now also U1.PD5; no longer U$1.PD5
- net GND: now also C10.1, C11.1, C12.1, C13.-, C14.-, C9.1, U1.GND@15, U1.GND@23, U1.GND@35, U1.GND@43, U1.PE2/!HWB, U1.UGND; no longer U$1.GND@15, U$1.GND@23, U$1.GND@35, U$1.GND@43, U$1.PE2/!HWB, U$1.UGND
- net HEARTBEAT: now also U1.PF5(ADC5); no longer U$1.PF5(ADC5)
- net LED1: now also U1.PF4(ADC4); no longer U$1.PF4(ADC4)
- net LED2: now also U1.PF1(ADC1); no longer U$1.PF1(ADC1)
- net LED3: now also U1.PF0(ADC0); no longer U$1.PF0(ADC0)
- net N$1: now also U1.UCAP; no longer U$1.UCAP
- net N$13: now also U1.XTAL2; no longer U$1.XTAL2
- net N$3: now also U1.XTAL1; no longer U$1.XTAL1
- net N$6: now also U1.D-; no longer U$1.D-
- net N$9: now also U1.D+; no longer U$1.D+
- net RST: now also U1.!RESET; no longer U$1.!RESET
- net RXLED: now also U1.PB0(SS); no longer U$1.PB0(SS)
- net SCLK: now also U1.PB1(SCK); no longer U$1.PB1(SCK)
- net SDATI: now also U1.PB2(MOSI); no longer U$1.PB2(MOSI)
- net SDATO: now also U1.PB3(MISO); no longer U$1.PB3(MISO)
- net VCC: now also C10.2, C11.2, C12.2, C9.2, U1.AREF, U1.AVCC@24, U1.AVCC@44, U1.UVCC, U1.VBUS, U1.VCC@14, U1.VCC@34; no longer U$1.AREF, U$1.AVCC@24, U$1.AVCC@44, U$1.UVCC, U$1.VBUS, U$1.VCC@14, U$1.VCC@34
- net VM: now also C13.+, C14.+
Other:
- moved on the sheet: C5, C6, C7, C8, R3, R6, R7, Y1
