File: Boards/PiEDB-Y16/Contingency/PDB/PDB.kicad_pcb (KiCad board)
At the start: 2 copper layers, 112.1 x 88.2 mm, 59 parts, among them J1 Conn_01x02, J2 Conn_01x04, J3 Conn_01x02, Q1 s8050_JSMSEMI, SW2 SW_SPDT, SW3 SW_MEC_5E, Sw1 D-SWITCH_MR5-111-C5N-BB, U2 CH340G, U3 PCF8574, Y1 12MHz

Commit message: Added to do for PDB
Parts:
- Converter1: value 5v_converter -> BUCK_CONVERTER_5V
Changed lines of the file:
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@@
     (fp_line (start 9.95 3.4) (end 9.95 -2.35)
       (stroke (width 0.1) (type solid)) (layer "F.Fab"))
-    (pad "1" thru_hole roundrect (at 0 0) (size 1.7 1.95) (drill 0.95) (layers "*.Cu" "*.Mask") (roundrect_rratio 0.1470588235)
+    (pad "1" thru_hole roundrect (at 0 0) (size 1.7 1.95) (drill 0.95) (layers "*.Cu" "*.Mask") (roundrect_rratio 0.147059)
       (net 19 "/Cell1+2+3") (pinfunction "Pin_3") (pintype "passive"))
     (pad "2" thru_hole oval (at 2.5 0) (size 1.7 1.95) (drill 0.95) (layers "*.Cu" "*.Mask")
@@
         (effects (font (size 1 1) (thickness 0.2)))
     )
-    (fp_text user "-" (at 6.05 2 unlocked) (layer "B.SilkS")
+    (fp_text user "+" (at -2.2 2.05 unlocked) (layer "B.SilkS")
         (effects (font (size 1 1) (thickness 0.2)) (justify mirror))
     )
-    (fp_text user "+" (at -2.2 2.05 unlocked) (layer "B.SilkS")
+    (fp_text user "-" (at 6.05 2 unlocked) (layer "B.SilkS")
         (effects (font (size 1 1) (thickness 0.2)) (justify mirror))
     )
@@
     (pad "24" thru_hole circle (at -13.97 -7.62 90) (size 1.6 1.6) (drill 1.1) (layers "*.Cu" "*.Mask")
       (net 52 "unconnected-(Pro1-RAW-Pad24)") (pinfunction "RAW") (pintype "power_out+no_connect"))
+    (model "D:/Users/Hsupe/Desktop/PiElectrical/Libraries/3dmodels/ARDUINO PRO MICRO.STEP"
+      (offset (xyz -14 -7.5 4))
+      (scale (xyz 1 1 1))
+      (rotate (xyz -90 0 0))
+    )
   )
   (footprint "PiE_Footprints:Fuse Holder SMD" (layer "F.Cu")
@@
         (effects (font (size 1 1) (thickness 0.2)) (justify mirror))
     )
-    (fp_text user "+" (at -6 2 unlocked) (layer "F.SilkS")
+    (fp_text user "-" (at 2 2 unlocked) (layer "F.SilkS")
         (effects (font (size 1 1) (thickness 0.2)))
     )
-    (fp_text user "-" (at 2 2 unlocked) (layer "F.SilkS")
+    (fp_text user "+" (at -6 2 unlocked) (layer "F.SilkS")
         (effects (font (size 1 1) (thickness 0.2)))
     )
@@
         (xy 0.354113 -0.320628)
       )
-      (stroke (width 0) (type solid)) (fill solid) (layer "F.Mask"))
+      (stroke (width 0) (type solid)) (fill solid) (layer "F.SilkS"))
     (fp_poly
       (pts
@@
         (xy 0.805929 -4.721218)
       )
-      (stroke (width 0) (type solid)) (fill solid) (layer "F.Mask"))
+      (stroke (width 0) (type solid)) (fill solid) (layer "F.SilkS"))
   )
   (footprint "Resistor_SMD:R_0603_1608Metric" (layer "F.Cu")
@@
         (effects (font (size 1 1) (thickness 0.2)))
     )
-    (fp_text user "-" (at 6.05 2 unlocked) (layer "B.SilkS")
+    (fp_text user "+" (at -2.2 2.05 unlocked) (layer "B.SilkS")
         (effects (font (size 1 1) (thickness 0.2)) (justify mirror))
     )
-    (fp_text user "+" (at -2.2 2.05 unlocked) (layer "B.SilkS")
+    (fp_text user "-" (at 6.05 2 unlocked) (layer "B.SilkS")
         (effects (font (size 1 1) (thickness 0.2)) (justify mirror))
     )
@@
         (effects (font (size 0.787402 0.787402) (thickness 0.15)))
     )
-    (fp_text value "5v_converter" (at 0 -26) (layer "F.Fab")
+    (fp_text value "BUCK_CONVERTER_5V" (at 0 -26) (layer "F.Fab")
         (effects (font (size 0.787402 0.787402) (thickness 0.15)))
     )
@@
         (effects (font (size 1.4 1.4) (thickness 0.15)))
     )
-    (fp_text user "OUT-" (at -2.794 -35.306) (layer "F.Fab")
-        (effects (font (size 1.4 1.4) (thickness 0.15)))
-    )
     (fp_text user "IN+" (at 9.906 -35.306) (layer "F.Fab")
         (effects (font (size 1.4 1.4) (thickness 0.15)))
     )
-    (fp_text user "OUT+" (at -9.144 -35.306) (layer "F.Fab")
+    (fp_text user "OUT-" (at -2.794 -35.306) (layer "F.Fab")
         (effects (font (size 1.4 1.4) (thickness 0.15)))
     )
@@
         (effects (font (size 1.4 1.4) (thickness 0.15)))
     )
+    (fp_text user "OUT+" (at -9.144 -35.306) (layer "F.Fab")
+        (effects (font (size 1.4 1.4) (thickness 0.15)))
+    )
     (fp_line (start -31.75 -17.78) (end -31.75 26.67)
       (stroke (width 0.127) (type solid)) (layer "F.SilkS"))
@@
         (effects (font (size 1 1) (thickness 0.2)))
     )
-    (fp_text user "+" (at -2.2 2.05 unlocked) (layer "B.SilkS")
+    (fp_text user "-" (at 6.05 2 unlocked) (layer "B.SilkS")
         (effects (font (size 1 1) (thickness 0.2)) (justify mirror))
     )
-    (fp_text user "-" (at 6.05 2 unlocked) (layer "B.SilkS")
+    (fp_text user "+" (at -2.2 2.05 unlocked) (layer "B.SilkS")
         (effects (font (size 1 1) (thickness 0.2)) (justify mirror))
     )
@@
         (effects (font (size 1 1) (thickness 0.15)))
     )
-    (pad "" np_thru_hole circle (at -0.05 5.1816) (size 3.24 3.24) (drill 3.24) (layers "F&B.Cu" "*.Mask"))
+    (pad "" np_thru_hole circle (at -0.05 0) (size 3.24 3.24) (drill 3.24) (layers "F&B.Cu" "*.Mask"))
   )
   (footprint "PiE_Footprints:PinHeader_1x04_P2.54mm_Vertical" (layer "F.Cu")
@@
     (style (thickness 0.15) (arrow_length 1.27) (text_position_mode 0) (extension_height 0.58642) (extension_offset 0.5) keep_text_aligned)
   )
+  (dimension (type orthogonal) (layer "Edge.Cuts")
+    (pts (xy 156.65 105.1) (xy 156.65 16.9))
+    (height 42.95)
+    (orientation 1)
+    (gr_text "88.2000 mm" (at 198.45 61 90) (layer "Edge.Cuts")
+      (effects (font (size 1 1) (thickness 0.15)))
+    )
+    (format (prefix "") (suffix "") (units 3) (units_format 1) (precision 4))
+    (style (thickness 0.1) (arrow_length 1.27) (text_position_mode 0) (extension_height 0.58642) (extension_offset 0.5) keep_text_aligned)
+  )
+  (dimension (type orthogonal) (layer "Edge.Cuts")
+    (pts (xy 98.35 60.05) (xy 98.3 105.1))
+    (height -63.2)
+    (orientation 1)
+    (gr_text "45.0500 mm" (at 34 82.575 90) (layer "Edge.Cuts")
+      (effects (font (size 1 1) (thickness 0.15)))
+    )
+    (format (prefix "") (suffix "") (units 3) (units_format 1) (precision 4))
+    (style (thickness 0.1) (arrow_length 1.27) (text_position_mode 0) (extension_height 0.58642) (extension_offset 0.5) keep_text_aligned)
+  )
   (segment (start 93.599 88.582) (end 93.599 91.568) (width 0.25) (layer "F.Cu") (net 1))
