File: Boards/PiEDB-Y17/gabesam board/gabesam board.kicad_pcb (KiCad board)
At the start: 2 copper layers, 109.5 x 59 mm, 25 parts, among them Q1 PMOS

Commit message: added 3D models and JLC footprints to buck test board
Parts:
- C1, C2, C_ADJ1, C_BYP1, C_IN1, C_OUT1, C_VCC1: footprint Capacitor_SMD:C_1206_3216Metric -> PCM_JLCPCB:C_1206
- R1, R_3, R_ADJ1, R_FB1, R_FB2, R_SEN1, R_T1: footprint Resistor_SMD:R_1206_3216Metric -> PCM_JLCPCB:R_1206
